Commit message: Rename package.

File: helix_description/urdf/dynamixel_block.xacro (robot description, xacro)
@@ -2,5 +2,5 @@
 <robot xmlns:xacro="http://ros.org/wiki/xacro">
 <!-- Import Rviz colors -->
-<xacro:include filename="$(find dynamixel_block_description)/urdf/dynamixel_block.material.xacro" />
+<xacro:include filename="$(find helix_description)/urdf/dynamixel_block.material.xacro" />
 <xacro:macro name="dynamixel_block" params="parent *origin">
   <joint name="origin_to_dynamixel_block" type="fixed">
@@ -19,5 +19,5 @@
       <origin xyz="0 0 0" rpy="0 0 0"/>
       <geometry>
-        <mesh filename="file://$(find dynamixel_block_description)/meshes/base_link.stl" scale="0.001 0.001 0.001"/>
+        <mesh filename="file://$(find helix_description)/meshes/base_link.stl" scale="0.001 0.001 0.001"/>
       </geometry>
       <material name="dynamixel_body"/>
@@ -26,5 +26,5 @@
       <origin xyz="0 0 0" rpy="0 0 0"/>
       <geometry>
-        <mesh filename="file://$(find dynamixel_block_description)/meshes/base_link.stl" scale="0.001 0.001 0.001"/>
+        <mesh filename="file://$(find helix_description)/meshes/base_link.stl" scale="0.001 0.001 0.001"/>
       </geometry>
     </collision>
@@ -39,5 +39,5 @@
       <origin xyz="-0.03 -0.037 -0.08475" rpy="0 0 0"/>
       <geometry>
-        <mesh filename="file://$(find dynamixel_block_description)/meshes/horn_0_1.stl" scale="0.001 0.001 0.001"/>
+        <mesh filename="file://$(find helix_description)/meshes/horn_0_1.stl" scale="0.001 0.001 0.001"/>
       </geometry>
       <material name="dynamixel_horn"/>
@@ -46,5 +46,5 @@
       <origin xyz="-0.03 -0.037 -0.08475" rpy="0 0 0"/>
       <geometry>
-        <mesh filename="file://$(find dynamixel_block_description)/meshes/horn_0_1.stl" scale="0.001 0.001 0.001"/>
+        <mesh filename="file://$(find helix_description)/meshes/horn_0_1.stl" scale="0.001 0.001 0.001"/>
       </geometry>
     </collision>
@@ -59,5 +59,5 @@
       <origin xyz="-0.03 -0.037 -0.01425" rpy="0 0 0"/>
       <geometry>
-        <mesh filename="file://$(find dynamixel_block_description)/meshes/horn_1_1.stl" scale="0.001 0.001 0.001"/>
+        <mesh filename="file://$(find helix_description)/meshes/horn_1_1.stl" scale="0.001 0.001 0.001"/>
       </geometry>
       <material name="dynamixel_horn"/>
@@ -66,5 +66,5 @@
       <origin xyz="-0.03 -0.037 -0.01425" rpy="0 0 0"/>
       <geometry>
-        <mesh filename="file://$(find dynamixel_block_description)/meshes/horn_1_1.stl" scale="0.001 0.001 0.001"/>
+        <mesh filename="file://$(find helix_description)/meshes/horn_1_1.stl" scale="0.001 0.001 0.001"/>
       </geometry>
     </collision>
@@ -79,5 +79,5 @@
       <origin xyz="-0.0 -0.037 -0.08475" rpy="0 0 0"/>
       <geometry>
-        <mesh filename="file://$(find dynamixel_block_description)/meshes/horn_2_1.stl" scale="0.001 0.001 0.001"/>
+        <mesh filename="file://$(find helix_description)/meshes/horn_2_1.stl" scale="0.001 0.001 0.001"/>
       </geometry>
       <material name="dynamixel_horn"/>
@@ -86,5 +86,5 @@
       <origin xyz="-0.0 -0.037 -0.08475" rpy="0 0 0"/>
       <geometry>
-        <mesh filename="file://$(find dynamixel_block_description)/meshes/horn_2_1.stl" scale="0.001 0.001 0.001"/>
+        <mesh filename="file://$(find helix_description)/meshes/horn_2_1.stl" scale="0.001 0.001 0.001"/>
       </geometry>
     </collision>
@@ -99,5 +99,5 @@
       <origin xyz="-0.0 -0.037 -0.01425" rpy="0 0 0"/>
       <geometry>
-        <mesh filename="file://$(find dynamixel_block_description)/meshes/horn_3_1.stl" scale="0.001 0.001 0.001"/>
+        <mesh filename="file://$(find helix_description)/meshes/horn_3_1.stl" scale="0.001 0.001 0.001"/>
       </geometry>
       <material name="dynamixel_horn"/>
@@ -106,5 +106,5 @@
       <origin xyz="-0.0 -0.037 -0.01425" rpy="0 0 0"/>
       <geometry>
-        <mesh filename="file://$(find dynamixel_block_description)/meshes/horn_3_1.stl" scale="0.001 0.001 0.001"/>
+        <mesh filename="file://$(find helix_description)/meshes/horn_3_1.stl" scale="0.001 0.001 0.001"/>
       </geometry>
     </collision>
@@ -119,5 +119,5 @@
       <origin xyz="0.03 -0.037 -0.08475" rpy="0 0 0"/>
       <geometry>
-        <mesh filename="file://$(find dynamixel_block_description)/meshes/horn_4_1.stl" scale="0.001 0.001 0.001"/>
+        <mesh filename="file://$(find helix_description)/meshes/horn_4_1.stl" scale="0.001 0.001 0.001"/>
       </geometry>
       <material name="dynamixel_horn"/>
@@ -126,5 +126,5 @@
       <origin xyz="0.03 -0.037 -0.08475" rpy="0 0 0"/>
       <geometry>
-        <mesh filename="file://$(find dynamixel_block_description)/meshes/horn_4_1.stl" scale="0.001 0.001 0.001"/>
+        <mesh filename="file://$(find helix_description)/meshes/horn_4_1.stl" scale="0.001 0.001 0.001"/>
       </geometry>
     </collision>
@@ -139,5 +139,5 @@
       <origin xyz="0.03 -0.037 -0.01425" rpy="0 0 0"/>
       <geometry>
-        <mesh filename="file://$(find dynamixel_block_description)/meshes/horn_5_1.stl" scale="0.001 0.001 0.001"/>
+        <mesh filename="file://$(find helix_description)/meshes/horn_5_1.stl" scale="0.001 0.001 0.001"/>
       </geometry>
       <material name="dynamixel_horn"/>
@@ -146,5 +146,5 @@
       <origin xyz="0.03 -0.037 -0.01425" rpy="0 0 0"/>
       <geometry>
-        <mesh filename="file://$(find dynamixel_block_description)/meshes/horn_5_1.stl" scale="0.001 0.001 0.001"/>
+        <mesh filename="file://$(find helix_description)/meshes/horn_5_1.stl" scale="0.001 0.001 0.001"/>
       </geometry>
     </collision>
@@ -159,5 +159,5 @@
       <origin xyz="0.03 0.037 -0.08475" rpy="0 0 0"/>
       <geometry>
-        <mesh filename="file://$(find dynamixel_block_description)/meshes/horn_6_1.stl" scale="0.001 0.001 0.001"/>
+        <mesh filename="file://$(find helix_description)/meshes/horn_6_1.stl" scale="0.001 0.001 0.001"/>
       </geometry>
       <material name="dynamixel_horn"/>
@@ -166,5 +166,5 @@
       <origin xyz="0.03 0.037 -0.08475" rpy="0 0 0"/>
       <geometry>
-        <mesh filename="file://$(find dynamixel_block_description)/meshes/horn_6_1.stl" scale="0.001 0.001 0.001"/>
+        <mesh filename="file://$(find helix_description)/meshes/horn_6_1.stl" scale="0.001 0.001 0.001"/>
       </geometry>
     </collision>
@@ -179,5 +179,5 @@
       <origin xyz="0.03 0.037 -0.01425" rpy="0 0 0"/>
       <geometry>
-        <mesh filename="file://$(find dynamixel_block_description)/meshes/horn_7_1.stl" scale="0.001 0.001 0.001"/>
+        <mesh filename="file://$(find helix_description)/meshes/horn_7_1.stl" scale="0.001 0.001 0.001"/>
       </geometry>
       <material name="dynamixel_horn"/>
@@ -186,5 +186,5 @@
       <origin xyz="0.03 0.037 -0.01425" rpy="0 0 0"/>
       <geometry>
-        <mesh filename="file://$(find dynamixel_block_description)/meshes/horn_7_1.stl" scale="0.001 0.001 0.001"/>
+        <mesh filename="file://$(find helix_description)/meshes/horn_7_1.stl" scale="0.001 0.001 0.001"/>
       </geometry>
     </collision>
@@ -199,5 +199,5 @@
       <origin xyz="-0.0 0.037 -0.08475" rpy="0 0 0"/>
       <geometry>
-        <mesh filename="file://$(find dynamixel_block_description)/meshes/horn_8_1.stl" scale="0.001 0.001 0.001"/>
+        <mesh filename="file://$(find helix_description)/meshes/horn_8_1.stl" scale="0.001 0.001 0.001"/>
       </geometry>
       <material name="dynamixel_horn"/>
@@ -206,5 +206,5 @@
       <origin xyz="-0.0 0.037 -0.08475" rpy="0 0 0"/>
       <geometry>
-        <mesh filename="file://$(find dynamixel_block_description)/meshes/horn_8_1.stl" scale="0.001 0.001 0.001"/>
+        <mesh filename="file://$(find helix_description)/meshes/horn_8_1.stl" scale="0.001 0.001 0.001"/>
       </geometry>
     </collision>
@@ -219,5 +219,5 @@
       <origin xyz="-0.0 0.037 -0.01425" rpy="0 0 0"/>
       <geometry>
-        <mesh filename="file://$(find dynamixel_block_description)/meshes/horn_9_1.stl" scale="0.001 0.001 0.001"/>
+        <mesh filename="file://$(find helix_description)/meshes/horn_9_1.stl" scale="0.001 0.001 0.001"/>
       </geometry>
       <material name="dynamixel_horn"/>
@@ -226,5 +226,5 @@
       <origin xyz="-0.0 0.037 -0.01425" rpy="0 0 0"/>
       <geometry>
-        <mesh filename="file://$(find dynamixel_block_description)/meshes/horn_9_1.stl" scale="0.001 0.001 0.001"/>
+        <mesh filename="file://$(find helix_description)/meshes/horn_9_1.stl" scale="0.001 0.001 0.001"/>
       </geometry>
     </collision>
@@ -239,5 +239,5 @@
       <origin xyz="-0.03 0.037 -0.08475" rpy="0 0 0"/>
       <geometry>
-        <mesh filename="file://$(find dynamixel_block_description)/meshes/horn_10_1.stl" scale="0.001 0.001 0.001"/>
+        <mesh filename="file://$(find helix_description)/meshes/horn_10_1.stl" scale="0.001 0.001 0.001"/>
       </geometry>
       <material name="dynamixel_horn"/>
@@ -246,5 +246,5 @@
       <origin xyz="-0.03 0.037 -0.08475" rpy="0 0 0"/>
       <geometry>
-        <mesh filename="file://$(find dynamixel_block_description)/meshes/horn_10_1.stl" scale="0.001 0.001 0.001"/>
+        <mesh filename="file://$(find helix_description)/meshes/horn_10_1.stl" scale="0.001 0.001 0.001"/>
       </geometry>
     </collision>
@@ -259,5 +259,5 @@
       <origin xyz="-0.03 0.037 -0.01425" rpy="0 0 0"/>
       <geometry>
-        <mesh filename="file://$(find dynamixel_block_description)/meshes/horn_11_1.stl" scale="0.001 0.001 0.001"/>
+        <mesh filename="file://$(find helix_description)/meshes/horn_11_1.stl" scale="0.001 0.001 0.001"/>
       </geometry>
       <material name="dynamixel_horn"/>
@@ -266,5 +266,5 @@
       <origin xyz="-0.03 0.037 -0.01425" rpy="0 0 0"/>
       <geometry>
-        <mesh filename="file://$(find dynamixel_block_description)/meshes/horn_11_1.stl" scale="0.001 0.001 0.001"/>
+        <mesh filename="file://$(find helix_description)/meshes/horn_11_1.stl" scale="0.001 0.001 0.001"/>
       </geometry>
     </collision>
@@ -355,5 +355,5 @@
       <origin xyz="0 0 0" rpy="0 0 0"/>
       <geometry>
-        <mesh filename="package://dynamixel_block_description/meshes/chain_link1.stl" scale="0.001 0.001 0.001"/>
+        <mesh filename="package://helix_description/meshes/chain_link1.stl" scale="0.001 0.001 0.001"/>
       </geometry>
       <material name="grey"/>
@@ -362,5 +362,5 @@
       <origin xyz="0 0 0" rpy="0 0 0"/>
       <geometry>
-        <mesh filename="package://dynamixel_block_description/meshes/chain_link1.stl" scale="0.001 0.001 0.001"/>
+        <mesh filename="package://helix_description/meshes/chain_link1.stl" scale="0.001 0.001 0.001"/>
       </geometry>
     </collision>
@@ -378,5 +378,5 @@
       <origin xyz="0 0 0.019" rpy="0 0 0"/>
       <geometry>
-        <mesh filename="package://dynamixel_block_description/meshes/chain_link2.stl" scale="0.001 0.001 0.001"/>
+        <mesh filename="package://helix_description/meshes/chain_link2.stl" scale="0.001 0.001 0.001"/>
       </geometry>
       <material name="grey"/>
@@ -385,5 +385,5 @@
       <origin xyz="0 0 0.019" rpy="0 0 0"/>
       <geometry>
-        <mesh filename="package://dynamixel_block_description/meshes/chain_link2.stl" scale="0.001 0.001 0.001"/>
+        <mesh filename="package://helix_description/meshes/chain_link2.stl" scale="0.001 0.001 0.001"/>
       </geometry>
     </collision>
@@ -409,5 +409,5 @@
       <origin xyz="0 0 0" rpy="0 0 0"/>
       <geometry>
-        <mesh filename="package://dynamixel_block_description/meshes/chain_link3.stl" scale="0.001 0.001 0.001"/>
+        <mesh filename="package://helix_description/meshes/chain_link3.stl" scale="0.001 0.001 0.001"/>
       </geometry>
       <material name="grey"/>
@@ -416,5 +416,5 @@
       <origin xyz="0 0 0" rpy="0 0 0"/>
       <geometry>
-        <mesh filename="package://dynamixel_block_description/meshes/chain_link3.stl" scale="0.001 0.001 0.001"/>
+        <mesh filename="package://helix_description/meshes/chain_link3.stl" scale="0.001 0.001 0.001"/>
       </geometry>
     </collision>
