Commit message: Add package:// and http:// option.

File: helix_description/urdf/dynamixel_block.xacro (robot description, xacro)
@@ -1,4 +1,5 @@
 <?xml version="1.0"?>
 <robot xmlns:xacro="http://ros.org/wiki/xacro">
+<xacro:arg name="mesh_url" default="package://helix_description" />
 <!-- Import Rviz colors -->
 <xacro:include filename="$(find helix_description)/urdf/dynamixel_block.material.xacro" />
@@ -19,5 +20,5 @@
       <origin xyz="0 0 0" rpy="0 0 0"/>
       <geometry>
-        <mesh filename="file://$(find helix_description)/meshes/base_link.stl" scale="0.001 0.001 0.001"/>
+        <mesh filename="$(arg mesh_url)/meshes/base_link.stl" scale="0.001 0.001 0.001"/>
       </geometry>
       <material name="dynamixel_body"/>
@@ -26,5 +27,5 @@
       <origin xyz="0 0 0" rpy="0 0 0"/>
       <geometry>
-        <mesh filename="file://$(find helix_description)/meshes/base_link.stl" scale="0.001 0.001 0.001"/>
+        <mesh filename="$(arg mesh_url)/meshes/base_link.stl" scale="0.001 0.001 0.001"/>
       </geometry>
     </collision>
@@ -39,5 +40,5 @@
       <origin xyz="-0.03 -0.037 -0.08475" rpy="0 0 0"/>
       <geometry>
-        <mesh filename="file://$(find helix_description)/meshes/horn_0_1.stl" scale="0.001 0.001 0.001"/>
+        <mesh filename="$(arg mesh_url)/meshes/horn_0_1.stl" scale="0.001 0.001 0.001"/>
       </geometry>
       <material name="dynamixel_horn"/>
@@ -46,5 +47,5 @@
       <origin xyz="-0.03 -0.037 -0.08475" rpy="0 0 0"/>
       <geometry>
-        <mesh filename="file://$(find helix_description)/meshes/horn_0_1.stl" scale="0.001 0.001 0.001"/>
+        <mesh filename="$(arg mesh_url)/meshes/horn_0_1.stl" scale="0.001 0.001 0.001"/>
       </geometry>
     </collision>
@@ -59,5 +60,5 @@
       <origin xyz="-0.03 -0.037 -0.01425" rpy="0 0 0"/>
       <geometry>
-        <mesh filename="file://$(find helix_description)/meshes/horn_1_1.stl" scale="0.001 0.001 0.001"/>
+        <mesh filename="$(arg mesh_url)/meshes/horn_1_1.stl" scale="0.001 0.001 0.001"/>
       </geometry>
       <material name="dynamixel_horn"/>
@@ -66,5 +67,5 @@
       <origin xyz="-0.03 -0.037 -0.01425" rpy="0 0 0"/>
       <geometry>
-        <mesh filename="file://$(find helix_description)/meshes/horn_1_1.stl" scale="0.001 0.001 0.001"/>
+        <mesh filename="$(arg mesh_url)/meshes/horn_1_1.stl" scale="0.001 0.001 0.001"/>
       </geometry>
     </collision>
@@ -79,5 +80,5 @@
       <origin xyz="-0.0 -0.037 -0.08475" rpy="0 0 0"/>
       <geometry>
-        <mesh filename="file://$(find helix_description)/meshes/horn_2_1.stl" scale="0.001 0.001 0.001"/>
+        <mesh filename="$(arg mesh_url)/meshes/horn_2_1.stl" scale="0.001 0.001 0.001"/>
       </geometry>
       <material name="dynamixel_horn"/>
@@ -86,5 +87,5 @@
       <origin xyz="-0.0 -0.037 -0.08475" rpy="0 0 0"/>
       <geometry>
-        <mesh filename="file://$(find helix_description)/meshes/horn_2_1.stl" scale="0.001 0.001 0.001"/>
+        <mesh filename="$(arg mesh_url)/meshes/horn_2_1.stl" scale="0.001 0.001 0.001"/>
       </geometry>
     </collision>
@@ -99,5 +100,5 @@
       <origin xyz="-0.0 -0.037 -0.01425" rpy="0 0 0"/>
       <geometry>
-        <mesh filename="file://$(find helix_description)/meshes/horn_3_1.stl" scale="0.001 0.001 0.001"/>
+        <mesh filename="$(arg mesh_url)/meshes/horn_3_1.stl" scale="0.001 0.001 0.001"/>
       </geometry>
       <material name="dynamixel_horn"/>
@@ -106,5 +107,5 @@
       <origin xyz="-0.0 -0.037 -0.01425" rpy="0 0 0"/>
       <geometry>
-        <mesh filename="file://$(find helix_description)/meshes/horn_3_1.stl" scale="0.001 0.001 0.001"/>
+        <mesh filename="$(arg mesh_url)/meshes/horn_3_1.stl" scale="0.001 0.001 0.001"/>
       </geometry>
     </collision>
@@ -119,5 +120,5 @@
       <origin xyz="0.03 -0.037 -0.08475" rpy="0 0 0"/>
       <geometry>
-        <mesh filename="file://$(find helix_description)/meshes/horn_4_1.stl" scale="0.001 0.001 0.001"/>
+        <mesh filename="$(arg mesh_url)/meshes/horn_4_1.stl" scale="0.001 0.001 0.001"/>
       </geometry>
       <material name="dynamixel_horn"/>
@@ -126,5 +127,5 @@
       <origin xyz="0.03 -0.037 -0.08475" rpy="0 0 0"/>
       <geometry>
-        <mesh filename="file://$(find helix_description)/meshes/horn_4_1.stl" scale="0.001 0.001 0.001"/>
+        <mesh filename="$(arg mesh_url)/meshes/horn_4_1.stl" scale="0.001 0.001 0.001"/>
       </geometry>
     </collision>
@@ -139,5 +140,5 @@
       <origin xyz="0.03 -0.037 -0.01425" rpy="0 0 0"/>
       <geometry>
-        <mesh filename="file://$(find helix_description)/meshes/horn_5_1.stl" scale="0.001 0.001 0.001"/>
+        <mesh filename="$(arg mesh_url)/meshes/horn_5_1.stl" scale="0.001 0.001 0.001"/>
       </geometry>
       <material name="dynamixel_horn"/>
@@ -146,5 +147,5 @@
       <origin xyz="0.03 -0.037 -0.01425" rpy="0 0 0"/>
       <geometry>
-        <mesh filename="file://$(find helix_description)/meshes/horn_5_1.stl" scale="0.001 0.001 0.001"/>
+        <mesh filename="$(arg mesh_url)/meshes/horn_5_1.stl" scale="0.001 0.001 0.001"/>
       </geometry>
     </collision>
@@ -159,5 +160,5 @@
       <origin xyz="0.03 0.037 -0.08475" rpy="0 0 0"/>
       <geometry>
-        <mesh filename="file://$(find helix_description)/meshes/horn_6_1.stl" scale="0.001 0.001 0.001"/>
+        <mesh filename="$(arg mesh_url)/meshes/horn_6_1.stl" scale="0.001 0.001 0.001"/>
       </geometry>
       <material name="dynamixel_horn"/>
@@ -166,5 +167,5 @@
       <origin xyz="0.03 0.037 -0.08475" rpy="0 0 0"/>
       <geometry>
-        <mesh filename="file://$(find helix_description)/meshes/horn_6_1.stl" scale="0.001 0.001 0.001"/>
+        <mesh filename="$(arg mesh_url)/meshes/horn_6_1.stl" scale="0.001 0.001 0.001"/>
       </geometry>
     </collision>
@@ -179,5 +180,5 @@
       <origin xyz="0.03 0.037 -0.01425" rpy="0 0 0"/>
       <geometry>
-        <mesh filename="file://$(find helix_description)/meshes/horn_7_1.stl" scale="0.001 0.001 0.001"/>
+        <mesh filename="$(arg mesh_url)/meshes/horn_7_1.stl" scale="0.001 0.001 0.001"/>
       </geometry>
       <material name="dynamixel_horn"/>
@@ -186,5 +187,5 @@
       <origin xyz="0.03 0.037 -0.01425" rpy="0 0 0"/>
       <geometry>
-        <mesh filename="file://$(find helix_description)/meshes/horn_7_1.stl" scale="0.001 0.001 0.001"/>
+        <mesh filename="$(arg mesh_url)/meshes/horn_7_1.stl" scale="0.001 0.001 0.001"/>
       </geometry>
     </collision>
@@ -199,5 +200,5 @@
       <origin xyz="-0.0 0.037 -0.08475" rpy="0 0 0"/>
       <geometry>
-        <mesh filename="file://$(find helix_description)/meshes/horn_8_1.stl" scale="0.001 0.001 0.001"/>
+        <mesh filename="$(arg mesh_url)/meshes/horn_8_1.stl" scale="0.001 0.001 0.001"/>
       </geometry>
       <material name="dynamixel_horn"/>
@@ -206,5 +207,5 @@
       <origin xyz="-0.0 0.037 -0.08475" rpy="0 0 0"/>
       <geometry>
-        <mesh filename="file://$(find helix_description)/meshes/horn_8_1.stl" scale="0.001 0.001 0.001"/>
+        <mesh filename="$(arg mesh_url)/meshes/horn_8_1.stl" scale="0.001 0.001 0.001"/>
       </geometry>
     </collision>
@@ -219,5 +220,5 @@
       <origin xyz="-0.0 0.037 -0.01425" rpy="0 0 0"/>
       <geometry>
-        <mesh filename="file://$(find helix_description)/meshes/horn_9_1.stl" scale="0.001 0.001 0.001"/>
+        <mesh filename="$(arg mesh_url)/meshes/horn_9_1.stl" scale="0.001 0.001 0.001"/>
       </geometry>
       <material name="dynamixel_horn"/>
@@ -226,5 +227,5 @@
       <origin xyz="-0.0 0.037 -0.01425" rpy="0 0 0"/>
       <geometry>
-        <mesh filename="file://$(find helix_description)/meshes/horn_9_1.stl" scale="0.001 0.001 0.001"/>
+        <mesh filename="$(arg mesh_url)/meshes/horn_9_1.stl" scale="0.001 0.001 0.001"/>
       </geometry>
     </collision>
@@ -239,5 +240,5 @@
       <origin xyz="-0.03 0.037 -0.08475" rpy="0 0 0"/>
       <geometry>
-        <mesh filename="file://$(find helix_description)/meshes/horn_10_1.stl" scale="0.001 0.001 0.001"/>
+        <mesh filename="$(arg mesh_url)/meshes/horn_10_1.stl" scale="0.001 0.001 0.001"/>
       </geometry>
       <material name="dynamixel_horn"/>
@@ -246,5 +247,5 @@
       <origin xyz="-0.03 0.037 -0.08475" rpy="0 0 0"/>
       <geometry>
-        <mesh filename="file://$(find helix_description)/meshes/horn_10_1.stl" scale="0.001 0.001 0.001"/>
+        <mesh filename="$(arg mesh_url)/meshes/horn_10_1.stl" scale="0.001 0.001 0.001"/>
       </geometry>
     </collision>
@@ -259,5 +260,5 @@
       <origin xyz="-0.03 0.037 -0.01425" rpy="0 0 0"/>
       <geometry>
-        <mesh filename="file://$(find helix_description)/meshes/horn_11_1.stl" scale="0.001 0.001 0.001"/>
+        <mesh filename="$(arg mesh_url)/meshes/horn_11_1.stl" scale="0.001 0.001 0.001"/>
       </geometry>
       <material name="dynamixel_horn"/>
@@ -266,5 +267,5 @@
       <origin xyz="-0.03 0.037 -0.01425" rpy="0 0 0"/>
       <geometry>
-        <mesh filename="file://$(find helix_description)/meshes/horn_11_1.stl" scale="0.001 0.001 0.001"/>
+        <mesh filename="$(arg mesh_url)/meshes/horn_11_1.stl" scale="0.001 0.001 0.001"/>
       </geometry>
     </collision>
@@ -342,89 +343,4 @@
     <axis xyz="0.0 -1.0 0.0"/>
   </joint>
-  <!-- Joint 1 -->
-  <!-- <joint name="dynamixel0to_delete" type="revolute">
-    <parent link="link1"/>
-    <child link="link2"/>
-    <origin xyz="0.012 0.0 0.017" rpy="0 0 0"/>
-    <axis xyz="0 0 1"/>
-    <limit velocity="4.8" effort="1" lower="-2.82743338823" upper="2.82743338823" />
-  </joint> -->
-  <!-- Link 1 -->
-  <!-- <link name="link1">
-    <visual>
-      <origin xyz="0 0 0" rpy="0 0 0"/>
-      <geometry>
-        <mesh filename="package://helix_description/meshes/chain_link1.stl" scale="0.001 0.001 0.001"/>
-      </geometry>
-      <material name="grey"/>
-    </visual>
-    <collision>
-      <origin xyz="0 0 0" rpy="0 0 0"/>
-      <geometry>
-        <mesh filename="package://helix_description/meshes/chain_link1.stl" scale="0.001 0.001 0.001"/>
-      </geometry>
-    </collision>
-    <inertial>
-      <origin xyz="3.0876154e-04 0.0000000e+00 -1.2176461e-04" />
-      <mass value="7.9119962e-02" />
-      <inertia ixx="1.2505234e-05" ixy="0.0" ixz="-1.7855208e-07"
-               iyy="2.1898364e-05" iyz="0.0"
-               izz="1.9267361e-05" />
-    </inertial>
-  </link> -->
-  <!--  Link 2 -->
-  <!-- <link name="link2">
-    <visual>
-      <origin xyz="0 0 0.019" rpy="0 0 0"/>
-      <geometry>
-        <mesh filename="package://helix_description/meshes/chain_link2.stl" scale="0.001 0.001 0.001"/>
-      </geometry>
-      <material name="grey"/>
-    </visual>
-    <collision>
-      <origin xyz="0 0 0.019" rpy="0 0 0"/>
-      <geometry>
-        <mesh filename="package://helix_description/meshes/chain_link2.stl" scale="0.001 0.001 0.001"/>
-      </geometry>
-    </collision>
-     <inertial>
-      <origin xyz="-3.0184870e-04 5.4043684e-04 0.047433464e-02" />
-      <mass value="9.8406837e-02" />
-      <inertia ixx="3.4543422e-05" ixy="-1.6031095e-08" ixz="-3.8375155e-07"
-               iyy="3.2689329e-05" iyz="2.8511935e-08"
-               izz="1.8850320e-05" />
-    </inertial>
-  </link> -->
-  <!--  Joint 2 -->
-  <!-- <joint name="dynamixel1" type="revolute">
-    <parent link="link2"/>
-    <child link="link3"/>
-    <origin xyz="0.0 0.0 0.0595" rpy="0 0 0"/>
-    <axis xyz="0 1 0"/>
-    <limit velocity="4.8" effort="1" lower="-1.79070781255" upper="1.57079632679" />
-  </joint> -->
-  <!--  Link 3 -->
-  <!-- <link name="link3">
-    <visual>
-      <origin xyz="0 0 0" rpy="0 0 0"/>
-      <geometry>
-        <mesh filename="package://helix_description/meshes/chain_link3.stl" scale="0.001 0.001 0.001"/>
-      </geometry>
-      <material name="grey"/>
-    </visual>
-    <collision>
-      <origin xyz="0 0 0" rpy="0 0 0"/>
-      <geometry>
-        <mesh filename="package://helix_description/meshes/chain_link3.stl" scale="0.001 0.001 0.001"/>
-      </geometry>
-    </collision>
-    <inertial>
-      <origin xyz="1.0308393e-02 3.7743363e-04 1.0170197e-01" />
-      <mass value="1.3850917e-01" />
-      <inertia ixx="3.3055381e-04" ixy="-9.7940978e-08" ixz="-3.8505711e-05"
-               iyy="3.4290447e-04" iyz="-1.5717516e-06"
-               izz="6.0346498e-05" />
-    </inertial>
-  </link> -->
 </xacro:macro>
 </robot>

File: helix_description/urdf/helix.urdf.xacro (robot description, xacro)
@@ -1,11 +1,8 @@
 <?xml version="1.0"?>
 <robot name="helix_description" xmlns:xacro="http://ros.org/wiki/xacro">
-  <!-- Uncomment this to show dynamixel!-->
   <xacro:include filename="$(find helix_description)/urdf/dynamixel_block.xacro" />
   <xacro:include filename="$(find helix_description)/urdf/dynamixel_block.ros2_control.xacro" />
-  <!-- Uncomment this to show hand!-->
-  <xacro:include filename="$(find helix_description)/urdf/helix.xacro" />
+  <xacro:include filename="$(find helix_description)/urdf/helix.xacro"  />
   <link name="world"/>
-  <!-- Uncomment this to show dynamixels!-->
   <xacro:dynamixel_block_ros2_control name="dynamixel_block_ros2_control" />
   <xacro:dynamixel_block parent="world">
