Commit message: Add package:// and http:// option.

File: helix_description/urdf/helix.xacro (robot description, xacro)
@@ -1,4 +1,5 @@
 <?xml version="1.0" ?>
 <robot name="URDF_Hand" xmlns:xacro="http://www.ros.org/wiki/xacro">
+<xacro:arg name="mesh_url" default="package://helix_description" />
 <xacro:include filename="$(find helix_description)/urdf/helix.materials.xacro" />
 <link name="base_link">
@@ -11,5 +12,5 @@
     <origin xyz="0 0 0" rpy="0 0 0"/>
     <geometry>
-      <mesh filename="file://$(find helix_description)/meshes/base_link.stl" scale="0.001 0.001 0.001"/>
+      <mesh filename="$(arg mesh_url)/meshes/base_link.stl" scale="0.001 0.001 0.001"/>
     </geometry>
     <material name="hand_base"/>
@@ -18,5 +19,5 @@
     <origin xyz="0 0 0" rpy="0 0 0"/>
     <geometry>
-      <mesh filename="file://$(find helix_description)/meshes/base_link.stl" scale="0.001 0.001 0.001"/>
+      <mesh filename="$(arg mesh_url)/meshes/base_link.stl" scale="0.001 0.001 0.001"/>
     </geometry>
   </collision>
@@ -31,5 +32,5 @@
     <origin xyz="-0.04166 -0.008898 -0.0855" rpy="0 0 0"/>
     <geometry>
-      <mesh filename="file://$(find helix_description)/meshes/Pinky_Base_1.stl" scale="0.001 0.001 0.001"/>
+      <mesh filename="$(arg mesh_url)/meshes/Pinky_Base_1.stl" scale="0.001 0.001 0.001"/>
     </geometry>
     <material name="finger_base"/>
@@ -38,5 +39,5 @@
     <origin xyz="-0.04166 -0.008898 -0.0855" rpy="0 0 0"/>
     <geometry>
-      <mesh filename="file://$(find helix_description)/meshes/Pinky_Base_1.stl" scale="0.001 0.001 0.001"/>
+      <mesh filename="$(arg mesh_url)/meshes/Pinky_Base_1.stl" scale="0.001 0.001 0.001"/>
     </geometry>
   </collision>
@@ -51,5 +52,5 @@
     <origin xyz="-0.019342 -0.005171 -0.0915" rpy="0 0 0"/>
     <geometry>
-      <mesh filename="file://$(find helix_description)/meshes/Ring_Base_1.stl" scale="0.001 0.001 0.001"/>
+      <mesh filename="$(arg mesh_url)/meshes/Ring_Base_1.stl" scale="0.001 0.001 0.001"/>
     </geometry>
     <material name="finger_base"/>
@@ -58,5 +59,5 @@
     <origin xyz="-0.019342 -0.005171 -0.0915" rpy="0 0 0"/>
     <geometry>
-      <mesh filename="file://$(find helix_description)/meshes/Ring_Base_1.stl" scale="0.001 0.001 0.001"/>
+      <mesh filename="$(arg mesh_url)/meshes/Ring_Base_1.stl" scale="0.001 0.001 0.001"/>
     </geometry>
   </collision>
@@ -71,5 +72,5 @@
     <origin xyz="0.003522 -0.0035 -0.0965" rpy="0 0 0"/>
     <geometry>
-      <mesh filename="file://$(find helix_description)/meshes/Middle_Base_1.stl" scale="0.001 0.001 0.001"/>
+      <mesh filename="$(arg mesh_url)/meshes/Middle_Base_1.stl" scale="0.001 0.001 0.001"/>
     </geometry>
     <material name="finger_base"/>
@@ -78,5 +79,5 @@
     <origin xyz="0.003522 -0.0035 -0.0965" rpy="0 0 0"/>
     <geometry>
-      <mesh filename="file://$(find helix_description)/meshes/Middle_Base_1.stl" scale="0.001 0.001 0.001"/>
+      <mesh filename="$(arg mesh_url)/meshes/Middle_Base_1.stl" scale="0.001 0.001 0.001"/>
     </geometry>
   </collision>
@@ -91,5 +92,5 @@
     <origin xyz="0.027097 -0.003767 -0.0915" rpy="0 0 0"/>
     <geometry>
-      <mesh filename="file://$(find helix_description)/meshes/Index_Base_1.stl" scale="0.001 0.001 0.001"/>
+      <mesh filename="$(arg mesh_url)/meshes/Index_Base_1.stl" scale="0.001 0.001 0.001"/>
     </geometry>
     <material name="finger_base"/>
@@ -98,5 +99,5 @@
     <origin xyz="0.027097 -0.003767 -0.0915" rpy="0 0 0"/>
     <geometry>
-      <mesh filename="file://$(find helix_description)/meshes/Index_Base_1.stl" scale="0.001 0.001 0.001"/>
+      <mesh filename="$(arg mesh_url)/meshes/Index_Base_1.stl" scale="0.001 0.001 0.001"/>
     </geometry>
   </collision>
@@ -111,5 +112,5 @@
     <origin xyz="-0.032646 -0.016381 -0.0971" rpy="0 0 0"/>
     <geometry>
-      <mesh filename="file://$(find helix_description)/meshes/Pinky_2dof_joint_1.stl" scale="0.001 0.001 0.001"/>
+      <mesh filename="$(arg mesh_url)/meshes/Pinky_2dof_joint_1.stl" scale="0.001 0.001 0.001"/>
     </geometry>
     <material name="2dof_joint"/>
@@ -118,5 +119,5 @@
     <origin xyz="-0.032646 -0.016381 -0.0971" rpy="0 0 0"/>
     <geometry>
-      <mesh filename="file://$(find helix_description)/meshes/Pinky_2dof_joint_1.stl" scale="0.001 0.001 0.001"/>
+      <mesh filename="$(arg mesh_url)/meshes/Pinky_2dof_joint_1.stl" scale="0.001 0.001 0.001"/>
     </geometry>
   </collision>
@@ -131,5 +132,5 @@
     <origin xyz="-0.011086 -0.013483 -0.1031" rpy="0 0 0"/>
     <geometry>
-      <mesh filename="file://$(find helix_description)/meshes/Ring_2dof_joint_1.stl" scale="0.001 0.001 0.001"/>
+      <mesh filename="$(arg mesh_url)/meshes/Ring_2dof_joint_1.stl" scale="0.001 0.001 0.001"/>
     </geometry>
     <material name="2dof_joint"/>
@@ -138,5 +139,5 @@
     <origin xyz="-0.011086 -0.013483 -0.1031" rpy="0 0 0"/>
     <geometry>
-      <mesh filename="file://$(find helix_description)/meshes/Ring_2dof_joint_1.stl" scale="0.001 0.001 0.001"/>
+      <mesh filename="$(arg mesh_url)/meshes/Ring_2dof_joint_1.stl" scale="0.001 0.001 0.001"/>
     </geometry>
   </collision>
@@ -151,5 +152,5 @@
     <origin xyz="0.011022 -0.0125 -0.1081" rpy="0 0 0"/>
     <geometry>
-      <mesh filename="file://$(find helix_description)/meshes/Middle_2dof_joint_1.stl" scale="0.001 0.001 0.001"/>
+      <mesh filename="$(arg mesh_url)/meshes/Middle_2dof_joint_1.stl" scale="0.001 0.001 0.001"/>
     </geometry>
     <material name="2dof_joint"/>
@@ -158,5 +159,5 @@
     <origin xyz="0.011022 -0.0125 -0.1081" rpy="0 0 0"/>
     <geometry>
-      <mesh filename="file://$(find helix_description)/meshes/Middle_2dof_joint_1.stl" scale="0.001 0.001 0.001"/>
+      <mesh filename="$(arg mesh_url)/meshes/Middle_2dof_joint_1.stl" scale="0.001 0.001 0.001"/>
     </geometry>
   </collision>
@@ -171,5 +172,5 @@
     <origin xyz="0.034116 -0.013147 -0.1031" rpy="0 0 0"/>
     <geometry>
-      <mesh filename="file://$(find helix_description)/meshes/Index_2dof_joint_1.stl" scale="0.001 0.001 0.001"/>
+      <mesh filename="$(arg mesh_url)/meshes/Index_2dof_joint_1.stl" scale="0.001 0.001 0.001"/>
     </geometry>
     <material name="2dof_joint"/>
@@ -178,5 +179,5 @@
     <origin xyz="0.034116 -0.013147 -0.1031" rpy="0 0 0"/>
     <geometry>
-      <mesh filename="file://$(find helix_description)/meshes/Index_2dof_joint_1.stl" scale="0.001 0.001 0.001"/>
+      <mesh filename="$(arg mesh_url)/meshes/Index_2dof_joint_1.stl" scale="0.001 0.001 0.001"/>
     </geometry>
   </collision>
@@ -191,5 +192,5 @@
     <origin xyz="-0.033283 -0.012939 -0.1061" rpy="0 0 0"/>
     <geometry>
-      <mesh filename="file://$(find helix_description)/meshes/Pinky_Proximal_1.stl" scale="0.001 0.001 0.001"/>
+      <mesh filename="$(arg mesh_url)/meshes/Pinky_Proximal_1.stl" scale="0.001 0.001 0.001"/>
     </geometry>
     <material name="proximal"/>
@@ -198,5 +199,5 @@
     <origin xyz="-0.033283 -0.012939 -0.1061" rpy="0 0 0"/>
     <geometry>
-      <mesh filename="file://$(find helix_description)/meshes/Pinky_Proximal_1.stl" scale="0.001 0.001 0.001"/>
+      <mesh filename="$(arg mesh_url)/meshes/Pinky_Proximal_1.stl" scale="0.001 0.001 0.001"/>
     </geometry>
   </collision>
@@ -211,5 +212,5 @@
     <origin xyz="-0.011391 -0.009996 -0.1121" rpy="0 0 0"/>
     <geometry>
-      <mesh filename="file://$(find helix_description)/meshes/Ring_Proximal_1.stl" scale="0.001 0.001 0.001"/>
+      <mesh filename="$(arg mesh_url)/meshes/Ring_Proximal_1.stl" scale="0.001 0.001 0.001"/>
     </geometry>
     <material name="proximal"/>
@@ -218,5 +219,5 @@
     <origin xyz="-0.011391 -0.009996 -0.1121" rpy="0 0 0"/>
     <geometry>
-      <mesh filename="file://$(find helix_description)/meshes/Ring_Proximal_1.stl" scale="0.001 0.001 0.001"/>
+      <mesh filename="$(arg mesh_url)/meshes/Ring_Proximal_1.stl" scale="0.001 0.001 0.001"/>
     </geometry>
   </collision>
@@ -231,5 +232,5 @@
     <origin xyz="0.011022 -0.009 -0.1171" rpy="0 0 0"/>
     <geometry>
-      <mesh filename="file://$(find helix_description)/meshes/Middle_Proximal_1.stl" scale="0.001 0.001 0.001"/>
+      <mesh filename="$(arg mesh_url)/meshes/Middle_Proximal_1.stl" scale="0.001 0.001 0.001"/>
     </geometry>
     <material name="proximal"/>
@@ -238,5 +239,5 @@
     <origin xyz="0.011022 -0.009 -0.1171" rpy="0 0 0"/>
     <geometry>
-      <mesh filename="file://$(find helix_description)/meshes/Middle_Proximal_1.stl" scale="0.001 0.001 0.001"/>
+      <mesh filename="$(arg mesh_url)/meshes/Middle_Proximal_1.stl" scale="0.001 0.001 0.001"/>
     </geometry>
   </collision>
@@ -251,5 +252,5 @@
     <origin xyz="0.034299 -0.009652 -0.1121" rpy="0 0 0"/>
     <geometry>
-      <mesh filename="file://$(find helix_description)/meshes/Index_Proximal_1.stl" scale="0.001 0.001 0.001"/>
+      <mesh filename="$(arg mesh_url)/meshes/Index_Proximal_1.stl" scale="0.001 0.001 0.001"/>
     </geometry>
     <material name="proximal"/>
@@ -258,5 +259,5 @@
     <origin xyz="0.034299 -0.009652 -0.1121" rpy="0 0 0"/>
     <geometry>
-      <mesh filename="file://$(find helix_description)/meshes/Index_Proximal_1.stl" scale="0.001 0.001 0.001"/>
+      <mesh filename="$(arg mesh_url)/meshes/Index_Proximal_1.stl" scale="0.001 0.001 0.001"/>
     </geometry>
   </collision>
@@ -271,5 +272,5 @@
     <origin xyz="0.03087 -0.016337 -0.03092" rpy="0 0 0"/>
     <geometry>
-      <mesh filename="file://$(find helix_description)/meshes/Thumb_Metacarpal_1.stl" scale="0.001 0.001 0.001"/>
+      <mesh filename="$(arg mesh_url)/meshes/Thumb_Metacarpal_1.stl" scale="0.001 0.001 0.001"/>
     </geometry>
     <material name="proximal"/>
@@ -278,5 +279,5 @@
     <origin xyz="0.03087 -0.016337 -0.03092" rpy="0 0 0"/>
     <geometry>
-      <mesh filename="file://$(find helix_description)/meshes/Thumb_Metacarpal_1.stl" scale="0.001 0.001 0.001"/>
+      <mesh filename="$(arg mesh_url)/meshes/Thumb_Metacarpal_1.stl" scale="0.001 0.001 0.001"/>
     </geometry>
   </collision>
@@ -291,5 +292,5 @@
     <origin xyz="-0.033283 -0.012939 -0.1446" rpy="0 0 0"/>
     <geometry>
-      <mesh filename="file://$(find helix_description)/meshes/Pinky_Middle_1.stl" scale="0.001 0.001 0.001"/>
+      <mesh filename="$(arg mesh_url)/meshes/Pinky_Middle_1.stl" scale="0.001 0.001 0.001"/>
     </geometry>
     <material name="middle"/>
@@ -298,5 +299,5 @@
     <origin xyz="-0.033283 -0.012939 -0.1446" rpy="0 0 0"/>
     <geometry>
-      <mesh filename="file://$(find helix_description)/meshes/Pinky_Middle_1.stl" scale="0.001 0.001 0.001"/>
+      <mesh filename="$(arg mesh_url)/meshes/Pinky_Middle_1.stl" scale="0.001 0.001 0.001"/>
     </geometry>
   </collision>
@@ -311,5 +312,5 @@
     <origin xyz="-0.011391 -0.009996 -0.1556" rpy="0 0 0"/>
     <geometry>
-      <mesh filename="file://$(find helix_description)/meshes/Ring_Middle_1.stl" scale="0.001 0.001 0.001"/>
+      <mesh filename="$(arg mesh_url)/meshes/Ring_Middle_1.stl" scale="0.001 0.001 0.001"/>
     </geometry>
     <material name="middle"/>
@@ -318,5 +319,5 @@
     <origin xyz="-0.011391 -0.009996 -0.1556" rpy="0 0 0"/>
     <geometry>
-      <mesh filename="file://$(find helix_description)/meshes/Ring_Middle_1.stl" scale="0.001 0.001 0.001"/>
+      <mesh filename="$(arg mesh_url)/meshes/Ring_Middle_1.stl" scale="0.001 0.001 0.001"/>
     </geometry>
   </collision>
@@ -331,5 +332,5 @@
     <origin xyz="0.011022 -0.009 -0.1656" rpy="0 0 0"/>
     <geometry>
-      <mesh filename="file://$(find helix_description)/meshes/Middle_Middle_1.stl" scale="0.001 0.001 0.001"/>
+      <mesh filename="$(arg mesh_url)/meshes/Middle_Middle_1.stl" scale="0.001 0.001 0.001"/>
     </geometry>
     <material name="middle"/>
@@ -338,5 +339,5 @@
     <origin xyz="0.011022 -0.009 -0.1656" rpy="0 0 0"/>
     <geometry>
-      <mesh filename="file://$(find helix_description)/meshes/Middle_Middle_1.stl" scale="0.001 0.001 0.001"/>
+      <mesh filename="$(arg mesh_url)/meshes/Middle_Middle_1.stl" scale="0.001 0.001 0.001"/>
     </geometry>
   </collision>
@@ -351,5 +352,5 @@
     <origin xyz="0.034299 -0.009652 -0.1556" rpy="0 0 0"/>
     <geometry>
-      <mesh filename="file://$(find helix_description)/meshes/Index_Middle_1.stl" scale="0.001 0.001 0.001"/>
+      <mesh filename="$(arg mesh_url)/meshes/Index_Middle_1.stl" scale="0.001 0.001 0.001"/>
     </geometry>
     <material name="middle"/>
@@ -358,5 +359,5 @@
     <origin xyz="0.034299 -0.009652 -0.1556" rpy="0 0 0"/>
     <geometry>
-      <mesh filename="file://$(find helix_description)/meshes/Index_Middle_1.stl" scale="0.001 0.001 0.001"/>
+      <mesh filename="$(arg mesh_url)/meshes/Index_Middle_1.stl" scale="0.001 0.001 0.001"/>
     </geometry>
   </collision>
@@ -371,5 +372,5 @@
     <origin xyz="0.055962 -0.013817 -0.074167" rpy="0 0 0"/>
     <geometry>
-      <mesh filename="file://$(find helix_description)/meshes/Thumb_Proximal_1.stl" scale="0.001 0.001 0.001"/>
+      <mesh filename="$(arg mesh_url)/meshes/Thumb_Proximal_1.stl" scale="0.001 0.001 0.001"/>
     </geometry>
     <material name="middle"/>
@@ -378,5 +379,5 @@
     <origin xyz="0.055962 -0.013817 -0.074167" rpy="0 0 0"/>
     <geometry>
-      <mesh filename="file://$(find helix_description)/meshes/Thumb_Proximal_1.stl" scale="0.001 0.001 0.001"/>
+      <mesh filename="$(arg mesh_url)/meshes/Thumb_Proximal_1.stl" scale="0.001 0.001 0.001"/>
     </geometry>
   </collision>
@@ -391,5 +392,5 @@
     <origin xyz="-0.033283 -0.012939 -0.1716" rpy="0 0 0"/>
     <geometry>
-      <mesh filename="file://$(find helix_description)/meshes/Pinky_Distal_1.stl" scale="0.001 0.001 0.001"/>
+      <mesh filename="$(arg mesh_url)/meshes/Pinky_Distal_1.stl" scale="0.001 0.001 0.001"/>
     </geometry>
     <material name="distal"/>
@@ -398,5 +399,5 @@
     <origin xyz="-0.033283 -0.012939 -0.1716" rpy="0 0 0"/>
     <geometry>
-      <mesh filename="file://$(find helix_description)/meshes/Pinky_Distal_1.stl" scale="0.001 0.001 0.001"/>
+      <mesh filename="$(arg mesh_url)/meshes/Pinky_Distal_1.stl" scale="0.001 0.001 0.001"/>
     </geometry>
   </collision>
@@ -411,5 +412,5 @@
     <origin xyz="-0.011391 -0.009996 -0.1876" rpy="0 0 0"/>
     <geometry>
-      <mesh filename="file://$(find helix_description)/meshes/Ring_Distal_1.stl" scale="0.001 0.001 0.001"/>
+      <mesh filename="$(arg mesh_url)/meshes/Ring_Distal_1.stl" scale="0.001 0.001 0.001"/>
     </geometry>
     <material name="distal"/>
@@ -418,5 +419,5 @@
     <origin xyz="-0.011391 -0.009996 -0.1876" rpy="0 0 0"/>
     <geometry>
-      <mesh filename="file://$(find helix_description)/meshes/Ring_Distal_1.stl" scale="0.001 0.001 0.001"/>
+      <mesh filename="$(arg mesh_url)/meshes/Ring_Distal_1.stl" scale="0.001 0.001 0.001"/>
     </geometry>
   </collision>
@@ -431,5 +432,5 @@
     <origin xyz="0.011022 -0.009 -0.2006" rpy="0 0 0"/>
     <geometry>
-      <mesh filename="file://$(find helix_description)/meshes/Middle_Distal_1.stl" scale="0.001 0.001 0.001"/>
+      <mesh filename="$(arg mesh_url)/meshes/Middle_Distal_1.stl" scale="0.001 0.001 0.001"/>
     </geometry>
     <material name="distal"/>
@@ -438,5 +439,5 @@
     <origin xyz="0.011022 -0.009 -0.2006" rpy="0 0 0"/>
     <geometry>
-      <mesh filename="file://$(find helix_description)/meshes/Middle_Distal_1.stl" scale="0.001 0.001 0.001"/>
+      <mesh filename="$(arg mesh_url)/meshes/Middle_Distal_1.stl" scale="0.001 0.001 0.001"/>
     </geometry>
   </collision>
@@ -451,5 +452,5 @@
     <origin xyz="0.034299 -0.009652 -0.1876" rpy="0 0 0"/>
     <geometry>
-      <mesh filename="file://$(find helix_description)/meshes/Index_Distal_1.stl" scale="0.001 0.001 0.001"/>
+      <mesh filename="$(arg mesh_url)/meshes/Index_Distal_1.stl" scale="0.001 0.001 0.001"/>
     </geometry>
     <material name="distal"/>
@@ -458,5 +459,5 @@
     <origin xyz="0.034299 -0.009652 -0.1876" rpy="0 0 0"/>
     <geometry>
-      <mesh filename="file://$(find helix_description)/meshes/Index_Distal_1.stl" scale="0.001 0.001 0.001"/>
+      <mesh filename="$(arg mesh_url)/meshes/Index_Distal_1.stl" scale="0.001 0.001 0.001"/>
     </geometry>
   </collision>
@@ -471,5 +472,5 @@
     <origin xyz="0.073263 -0.013776 -0.104592" rpy="0 0 0"/>
     <geometry>
-      <mesh filename="file://$(find helix_description)/meshes/Thumb_Distal_1.stl" scale="0.001 0.001 0.001"/>
+      <mesh filename="$(arg mesh_url)/meshes/Thumb_Distal_1.stl" scale="0.001 0.001 0.001"/>
     </geometry>
     <material name="distal"/>
@@ -478,5 +479,5 @@
     <origin xyz="0.073263 -0.013776 -0.104592" rpy="0 0 0"/>
     <geometry>
-      <mesh filename="file://$(find helix_description)/meshes/Thumb_Distal_1.stl" scale="0.001 0.001 0.001"/>
+      <mesh filename="$(arg mesh_url)/meshes/Thumb_Distal_1.stl" scale="0.001 0.001 0.001"/>
     </geometry>
   </collision>
@@ -491,5 +492,5 @@
     <origin xyz="0.018032 -0.003966 -0.045336" rpy="0 0 0"/>
     <geometry>
-      <mesh filename="file://$(find helix_description)/meshes/Thumb_Base_1.stl" scale="0.001 0.001 0.001"/>
+      <mesh filename="$(arg mesh_url)/meshes/Thumb_Base_1.stl" scale="0.001 0.001 0.001"/>
     </geometry>
     <material name="finger_base"/>
@@ -498,5 +499,5 @@
     <origin xyz="0.018032 -0.003966 -0.045336" rpy="0 0 0"/>
     <geometry>
-      <mesh filename="file://$(find helix_description)/meshes/Thumb_Base_1.stl" scale="0.001 0.001 0.001"/>
+      <mesh filename="$(arg mesh_url)/meshes/Thumb_Base_1.stl" scale="0.001 0.001 0.001"/>
     </geometry>
   </collision>
@@ -511,5 +512,5 @@
     <origin xyz="0.026985 -0.012128 -0.043132" rpy="0 0 0"/>
     <geometry>
-      <mesh filename="file://$(find helix_description)/meshes/Thumb_2dof_joint_1.stl" scale="0.001 0.001 0.001"/>
+      <mesh filename="$(arg mesh_url)/meshes/Thumb_2dof_joint_1.stl" scale="0.001 0.001 0.001"/>
     </geometry>
     <material name="2dof_joint"/>
@@ -518,5 +519,5 @@
     <origin xyz="0.026985 -0.012128 -0.043132" rpy="0 0 0"/>
     <geometry>
-      <mesh filename="file://$(find helix_description)/meshes/Thumb_2dof_joint_1.stl" scale="0.001 0.001 0.001"/>
+      <mesh filename="$(arg mesh_url)/meshes/Thumb_2dof_joint_1.stl" scale="0.001 0.001 0.001"/>
     </geometry>
   </collision>
