Commit message: Improve description during dummy mode testing Use more descriptive naming Include placeholder urdf for arm Add rviz config

File: helix_description/urdf/helix.urdf.xacro (robot description, xacro)
@@ -3,15 +3,14 @@
   <xacro:include filename="$(find helix_description)/urdf/motor_head.xacro" />
   <xacro:include filename="$(find helix_description)/urdf/helix.ros2_control.xacro" />
-  <!-- <xacro:include filename="$(find helix_description)/urdf/helix.xacro"  /> -->
-  <link name="world"/>
+  <xacro:include filename="$(find helix_description)/urdf/helix_arm.xacro"  />
+  <link name="origin"/>
   <xacro:helix_ros2_control name="helix_ros2_control" />
-  <xacro:motor_head parent="world">
+  <xacro:motor_head parent="origin">
     <origin xyz="0 0 0" rpy="0 0 0" />
   </xacro:motor_head>
-<!--
-  <joint name="motor_head_to_world" type="fixed">
-    <origin xyz="0.0 0.0 0.1" rpy="0 0 0"/>
-    <parent link="world"/>
-    <child link="base"/>
-  </joint> -->
+  <joint name="arm_to_origin" type="fixed">
+    <origin xyz="0.0 0.0 0.0" rpy="3.14 0 0"/>
+    <parent link="origin"/>
+    <child link="Index_Base_1"/>
+  </joint>
 </robot>

File: helix_description/urdf/helix_arm.xacro (robot description, xacro)
@@ -3,83 +3,106 @@
 <!-- URDF Representing the Helix arm -->
 <xacro:arg name="mesh_url" default="package://helix_description" />
-<xacro:include filename="$(find helix_description)/urdf/helix.materials.xacro" />
-<link name="base_link">
+<xacro:include filename="$(find helix_description)/urdf/helix_arm.materials.xacro" />
+<!-- Example below for a rigid serial chain. Maybe not relevant at all for flexible Helix arm representation. -->
+<link name="Index_Base_1">
   <inertial>
-    <origin xyz="-0.0005471831423920315 -0.0016798569855821554 0.04631267638063307" rpy="0 0 0"/>
-    <mass value="0.40903933360000916"/>
-    <inertia ixx="0.000261" iyy="0.00052" izz="0.000266" ixy="-0.0" iyz="-1.4e-05" ixz="-5e-06"/>
+    <origin xyz="-0.007201714291713072 0.005885230272430774 0.0016787722912366132" rpy="0 0 0"/>
+    <mass value="0.01722650129403022"/>
+    <inertia ixx="1e-06" iyy="1e-06" izz="1e-06" ixy="0.0" iyz="0.0" ixz="-0.0"/>
   </inertial>
   <visual>
-    <origin xyz="0 0 0" rpy="0 0 0"/>
+    <origin xyz="0.027097 -0.003767 -0.0915" rpy="0 0 0"/>
     <geometry>
-      <mesh filename="$(arg mesh_url)/meshes/base_link.stl" scale="0.001 0.001 0.001"/>
+      <mesh filename="$(arg mesh_url)/meshes/Index_Base_1.stl" scale="0.001 0.001 0.001"/>
     </geometry>
-    <material name="hand_base"/>
+    <material name="finger_base"/>
   </visual>
   <collision>
-    <origin xyz="0 0 0" rpy="0 0 0"/>
+    <origin xyz="0.027097 -0.003767 -0.0915" rpy="0 0 0"/>
     <geometry>
-      <mesh filename="$(arg mesh_url)/meshes/base_link.stl" scale="0.001 0.001 0.001"/>
+      <mesh filename="$(arg mesh_url)/meshes/Index_Base_1.stl" scale="0.001 0.001 0.001"/>
     </geometry>
   </collision>
 </link>
-<link name="Thumb_2dof_joint_1">
+<link name="Index_2dof_joint_1">
   <inertial>
-    <origin xyz="-0.0009098329677024661 0.001066944068375937 -0.010524206941038762" rpy="0 0 0"/>
-    <mass value="0.014036293256380273"/>
-    <inertia ixx="1e-06" iyy="2e-06" izz="1e-06" ixy="0.0" iyz="0.0" ixz="0.0"/>
+    <origin xyz="-0.001481711245915833 -0.0034266921818958945 0.0028828067230253634" rpy="0 0 0"/>
+    <mass value="0.0074922865960129585"/>
+    <inertia ixx="0.0" iyy="0.0" izz="0.0" ixy="0.0" iyz="-0.0" ixz="0.0"/>
   </inertial>
   <visual>
-    <origin xyz="0.026985 -0.012128 -0.043132" rpy="0 0 0"/>
+    <origin xyz="0.034116 -0.013147 -0.1031" rpy="0 0 0"/>
     <geometry>
-      <mesh filename="$(arg mesh_url)/meshes/Thumb_2dof_joint_1.stl" scale="0.001 0.001 0.001"/>
+      <mesh filename="$(arg mesh_url)/meshes/Index_2dof_joint_1.stl" scale="0.001 0.001 0.001"/>
     </geometry>
     <material name="2dof_joint"/>
   </visual>
   <collision>
-    <origin xyz="0.026985 -0.012128 -0.043132" rpy="0 0 0"/>
+    <origin xyz="0.034116 -0.013147 -0.1031" rpy="0 0 0"/>
     <geometry>
-      <mesh filename="$(arg mesh_url)/meshes/Thumb_2dof_joint_1.stl" scale="0.001 0.001 0.001"/>
+      <mesh filename="$(arg mesh_url)/meshes/Index_2dof_joint_1.stl" scale="0.001 0.001 0.001"/>
     </geometry>
   </collision>
 </link>
-<joint name="Pinky_Base" type="fixed">
-  <origin xyz="0.04166 0.008898 0.0855" rpy="0 0 0"/>
-  <parent link="base_link"/>
-  <child link="Pinky_Base_1"/>
-</joint>
-<joint name="Ring_Base" type="fixed">
-  <origin xyz="0.019342 0.005171 0.0915" rpy="0 0 0"/>
-  <parent link="base_link"/>
-  <child link="Ring_Base_1"/>
-</joint>
-<joint name="Middle_Base" type="fixed">
-  <origin xyz="-0.003522 0.0035 0.0965" rpy="0 0 0"/>
-  <parent link="base_link"/>
-  <child link="Middle_Base_1"/>
-</joint>
-<joint name="Index_Base" type="fixed">
-  <origin xyz="-0.027097 0.003767 0.0915" rpy="0 0 0"/>
-  <parent link="base_link"/>
-  <child link="Index_Base_1"/>
-</joint>
-<joint name="Pinky_MCP_Orth" type="continuous">
-  <origin xyz="-0.009014 0.007483 0.0116" rpy="0 0 0"/>
-  <parent link="Pinky_Base_1"/>
-  <child link="Pinky_2dof_joint_1"/>
-  <axis xyz="-0.182236 0.983255 0.0"/>
-</joint>
-<joint name="Ring_MCP_Orth" type="continuous">
-  <origin xyz="-0.008256 0.008312 0.0116" rpy="0 0 0"/>
-  <parent link="Ring_Base_1"/>
-  <child link="Ring_2dof_joint_1"/>
-  <axis xyz="-0.087156 0.996195 0.0"/>
-</joint>
-<joint name="Middle_MCP_Orth" type="continuous">
-  <origin xyz="-0.0075 0.009 0.0116" rpy="0 0 0"/>
-  <parent link="Middle_Base_1"/>
-  <child link="Middle_2dof_joint_1"/>
-  <axis xyz="-0.0 1.0 0.0"/>
-</joint>
+<link name="Index_Proximal_1">
+  <inertial>
+    <origin xyz="0.0006445383282672051 0.001274183043787739 0.021749999999999825" rpy="0 0 0"/>
+    <mass value="0.039861235764857395"/>
+    <inertia ixx="5e-06" iyy="6e-06" izz="1e-06" ixy="0.0" iyz="-0.0" ixz="0.0"/>
+  </inertial>
+  <visual>
+    <origin xyz="0.034299 -0.009652 -0.1121" rpy="0 0 0"/>
+    <geometry>
+      <mesh filename="$(arg mesh_url)/meshes/Index_Proximal_1.stl" scale="0.001 0.001 0.001"/>
+    </geometry>
+    <material name="proximal"/>
+  </visual>
+  <collision>
+    <origin xyz="0.034299 -0.009652 -0.1121" rpy="0 0 0"/>
+    <geometry>
+      <mesh filename="$(arg mesh_url)/meshes/Index_Proximal_1.stl" scale="0.001 0.001 0.001"/>
+    </geometry>
+  </collision>
+</link>
+<link name="Index_Middle_1">
+  <inertial>
+    <origin xyz="-0.000786432090189769 0.0012174084476994501 0.015999999999999903" rpy="0 0 0"/>
+    <mass value="0.02706545369444013"/>
+    <inertia ixx="2e-06" iyy="2e-06" izz="1e-06" ixy="-0.0" iyz="0.0" ixz="0.0"/>
+  </inertial>
+  <visual>
+    <origin xyz="0.034299 -0.009652 -0.1556" rpy="0 0 0"/>
+    <geometry>
+      <mesh filename="$(arg mesh_url)/meshes/Index_Middle_1.stl" scale="0.001 0.001 0.001"/>
+    </geometry>
+    <material name="middle"/>
+  </visual>
+  <collision>
+    <origin xyz="0.034299 -0.009652 -0.1556" rpy="0 0 0"/>
+    <geometry>
+      <mesh filename="$(arg mesh_url)/meshes/Index_Middle_1.stl" scale="0.001 0.001 0.001"/>
+    </geometry>
+  </collision>
+</link>
+<link name="Index_Distal_1">
+  <inertial>
+    <origin xyz="0.0006324531075937584 0.0009652221564475042 0.012319161138346219" rpy="0 0 0"/>
+    <mass value="0.019789884505209417"/>
+    <inertia ixx="1e-06" iyy="1e-06" izz="0.0" ixy="0.0" iyz="-0.0" ixz="0.0"/>
+  </inertial>
+  <visual>
+    <origin xyz="0.034299 -0.009652 -0.1876" rpy="0 0 0"/>
+    <geometry>
+      <mesh filename="$(arg mesh_url)/meshes/Index_Distal_1.stl" scale="0.001 0.001 0.001"/>
+    </geometry>
+    <material name="distal"/>
+  </visual>
+  <collision>
+    <origin xyz="0.034299 -0.009652 -0.1876" rpy="0 0 0"/>
+    <geometry>
+      <mesh filename="$(arg mesh_url)/meshes/Index_Distal_1.stl" scale="0.001 0.001 0.001"/>
+    </geometry>
+  </collision>
+</link>
 <joint name="Index_MCP_Orth" type="continuous">
   <origin xyz="-0.007019 0.00938 0.0116" rpy="0 0 0"/>
@@ -87,22 +110,4 @@
   <child link="Index_2dof_joint_1"/>
   <axis xyz="0.052336 0.99863 0.0"/>
-</joint>
-<joint name="Pinky_MCP" type="continuous">
-  <origin xyz="0.000637 -0.003442 0.009" rpy="0 0 0"/>
-  <parent link="Pinky_2dof_joint_1"/>
-  <child link="Pinky_Proximal_1"/>
-  <axis xyz="-0.983255 -0.182236 -0.0"/>
-</joint>
-<joint name="Ring_MCP" type="continuous">
-  <origin xyz="0.000305 -0.003487 0.009" rpy="0 0 0"/>
-  <parent link="Ring_2dof_joint_1"/>
-  <child link="Ring_Proximal_1"/>
-  <axis xyz="-0.996195 -0.087156 -0.0"/>
-</joint>
-<joint name="Middle_MCP" type="continuous">
-  <origin xyz="0.0 -0.0035 0.009" rpy="0 0 0"/>
-  <parent link="Middle_2dof_joint_1"/>
-  <child link="Middle_Proximal_1"/>
-  <axis xyz="-1.0 0.0 -0.0"/>
 </joint>
 <joint name="Index_MCP" type="continuous">
@@ -112,28 +117,4 @@
   <axis xyz="-0.99863 0.052336 -0.0"/>
 </joint>
-<joint name="Thumb_CMC_Orth" type="continuous">
-  <origin xyz="-0.003885 0.004209 -0.012212" rpy="0 0 0"/>
-  <parent link="Thumb_2dof_joint_1"/>
-  <child link="Thumb_Metacarpal_1"/>
-  <axis xyz="-0.150384 -0.984808 -0.086824"/>
-</joint>
-<joint name="Pinky_PIP" type="continuous">
-  <origin xyz="0.0 0.0 0.0385" rpy="0 0 0"/>
-  <parent link="Pinky_Proximal_1"/>
-  <child link="Pinky_Middle_1"/>
-  <axis xyz="-0.983255 -0.182236 0.0"/>
-</joint>
-<joint name="Ring_PIP" type="continuous">
-  <origin xyz="0.0 0.0 0.0435" rpy="0 0 0"/>
-  <parent link="Ring_Proximal_1"/>
-  <child link="Ring_Middle_1"/>
-  <axis xyz="-0.996195 -0.087156 0.0"/>
-</joint>
-<joint name="Middle_PIP" type="continuous">
-  <origin xyz="0.0 0.0 0.0485" rpy="0 0 0"/>
-  <parent link="Middle_Proximal_1"/>
-  <child link="Middle_Middle_1"/>
-  <axis xyz="-1.0 -0.0 0.0"/>
-</joint>
 <joint name="Index_PIP" type="continuous">
   <origin xyz="0.0 0.0 0.0435" rpy="0 0 0"/>
@@ -141,28 +122,4 @@
   <child link="Index_Middle_1"/>
   <axis xyz="-0.99863 0.052336 0.0"/>
-</joint>
-<joint name="Thumb_MCP" type="continuous">
-  <origin xyz="-0.025092 -0.00252 0.043247" rpy="0 0 0"/>
-  <parent link="Thumb_Metacarpal_1"/>
-  <child link="Thumb_Proximal_1"/>
-  <axis xyz="-0.788081 0.422615 -0.447577"/>
-</joint>
-<joint name="Pinky_DIP" type="continuous">
-  <origin xyz="0.0 0.0 0.027" rpy="0 0 0"/>
-  <parent link="Pinky_Middle_1"/>
-  <child link="Pinky_Distal_1"/>
-  <axis xyz="-0.983255 -0.182236 0.0"/>
-</joint>
-<joint name="Ring_DIP" type="continuous">
-  <origin xyz="0.0 0.0 0.032" rpy="0 0 0"/>
-  <parent link="Ring_Middle_1"/>
-  <child link="Ring_Distal_1"/>
-  <axis xyz="-0.996195 -0.087156 0.0"/>
-</joint>
-<joint name="Middle_DIP" type="continuous">
-  <origin xyz="0.0 0.0 0.035" rpy="0 0 0"/>
-  <parent link="Middle_Middle_1"/>
-  <child link="Middle_Distal_1"/>
-  <axis xyz="-1.0 -0.0 0.0"/>
 </joint>
 <joint name="Index_DIP" type="continuous">
@@ -172,20 +129,3 @@
   <axis xyz="-0.99863 0.052336 0.0"/>
 </joint>
-<joint name="Thumb_IP" type="continuous">
-  <origin xyz="-0.017301 -4.1e-05 0.030425" rpy="0 0 0"/>
-  <parent link="Thumb_Proximal_1"/>
-  <child link="Thumb_Distal_1"/>
-  <axis xyz="-0.788081 0.422615 -0.447577"/>
-</joint>
-<joint name="Thumb_Base" type="fixed">
-  <origin xyz="-0.018032 0.003966 0.045336" rpy="0 0 0"/>
-  <parent link="base_link"/>
-  <child link="Thumb_Base_1"/>
-</joint>
-<joint name="Thumb_CMC" type="continuous">
-  <origin xyz="-0.008953 0.008162 -0.002204" rpy="0 0 0"/>
-  <parent link="Thumb_Base_1"/>
-  <child link="Thumb_2dof_joint_1"/>
-  <axis xyz="0.494314 0.001155 -0.869283"/>
-</joint>
 </robot>

File: helix_description/urdf/motor_head.materials.xacro (robot description, xacro)
@@ -1,6 +1,6 @@
 <?xml version="1.0"?>
 <robot>
-  <material name="dynamixel_horn">
-    <color rgba="0.7 0.6 0.0 1.000"/>
+  <material name="black">
+    <color rgba="0.2 0.2 0.2 1.0"/>
   </material>
   <material name='clear'>

File: helix_description/urdf/motor_head.xacro (robot description, xacro)
@@ -36,4 +36,5 @@
   </link>
   <!-- Joint 0 -->
+  <!-- TODO check changing to continuous, removing limits -->
   <joint name="joint0" type="revolute">
     <parent link="base"/>
@@ -48,7 +49,7 @@
       <origin xyz="0 0 0" rpy="0 1.57 0"/>
       <geometry>
-        <mesh filename="$(arg mesh_url)/meshes/horn_0_1.stl" scale="0.001 0.001 0.001"/>
-      </geometry>
-      <material name="dynamixel_horn"/>
+        <cylinder length="0.015" radius="0.02"/>
+      </geometry>
+      <material name="black"/>
     </visual>
   </link>
@@ -66,7 +67,7 @@
       <origin xyz="0 0 0" rpy="0 1.57 0"/>
       <geometry>
-        <mesh filename="$(arg mesh_url)/meshes/horn_0_1.stl" scale="0.001 0.001 0.001"/>
-      </geometry>
-      <material name="dynamixel_horn"/>
+        <cylinder length="0.015" radius="0.02"/>
+      </geometry>
+      <material name="black"/>
     </visual>
   </link>
@@ -84,7 +85,7 @@
       <origin xyz="0 0 0" rpy="0 1.57 0"/>
       <geometry>
-        <mesh filename="$(arg mesh_url)/meshes/horn_0_1.stl" scale="0.001 0.001 0.001"/>
-      </geometry>
-      <material name="dynamixel_horn"/>
+        <cylinder length="0.015" radius="0.02"/>
+      </geometry>
+      <material name="black"/>
     </visual>
   </link>
@@ -102,7 +103,7 @@
       <origin xyz="0 0 0" rpy="0 1.57 0"/>
       <geometry>
-        <mesh filename="$(arg mesh_url)/meshes/horn_0_1.stl" scale="0.001 0.001 0.001"/>
-      </geometry>
-      <material name="dynamixel_horn"/>
+        <cylinder length="0.015" radius="0.02"/>
+      </geometry>
+      <material name="black"/>
     </visual>
   </link>
@@ -120,7 +121,7 @@
       <origin xyz="0 0 0" rpy="0 1.57 0"/>
       <geometry>
-        <mesh filename="$(arg mesh_url)/meshes/horn_0_1.stl" scale="0.001 0.001 0.001"/>
-      </geometry>
-      <material name="dynamixel_horn"/>
+        <cylinder length="0.015" radius="0.02"/>
+      </geometry>
+      <material name="black"/>
     </visual>
   </link>
@@ -138,7 +139,7 @@
       <origin xyz="0 0 0" rpy="0 1.57 0"/>
       <geometry>
-        <mesh filename="$(arg mesh_url)/meshes/horn_0_1.stl" scale="0.001 0.001 0.001"/>
-      </geometry>
-      <material name="dynamixel_horn"/>
+        <cylinder length="0.015" radius="0.02"/>
+      </geometry>
+      <material name="black"/>
     </visual>
   </link>
@@ -156,7 +157,7 @@
       <origin xyz="0 0 0" rpy="0 1.57 0"/>
       <geometry>
-        <mesh filename="$(arg mesh_url)/meshes/horn_0_1.stl" scale="0.001 0.001 0.001"/>
-      </geometry>
-      <material name="dynamixel_horn"/>
+        <cylinder length="0.015" radius="0.02"/>
+      </geometry>
+      <material name="black"/>
     </visual>
   </link>
@@ -174,7 +175,7 @@
       <origin xyz="0 0 0" rpy="0 1.57 0"/>
       <geometry>
-        <mesh filename="$(arg mesh_url)/meshes/horn_0_1.stl" scale="0.001 0.001 0.001"/>
-      </geometry>
-      <material name="dynamixel_horn"/>
+        <cylinder length="0.015" radius="0.02"/>
+      </geometry>
+      <material name="black"/>
     </visual>
   </link>
@@ -192,7 +193,7 @@
       <origin xyz="0 0 0" rpy="0 1.57 0"/>
       <geometry>
-        <mesh filename="$(arg mesh_url)/meshes/horn_0_1.stl" scale="0.001 0.001 0.001"/>
-      </geometry>
-      <material name="dynamixel_horn"/>
+        <cylinder length="0.015" radius="0.02"/>
+      </geometry>
+      <material name="black"/>
     </visual>
   </link>

Commit message: Add floating segment end discs to URDF for arm visualisation

File: helix_description/urdf/helix.urdf.xacro (robot description, xacro)
@@ -10,7 +10,7 @@
   </xacro:motor_head>
   <joint name="arm_to_origin" type="fixed">
-    <origin xyz="0.0 0.0 0.0" rpy="3.14 0 0"/>
+    <origin xyz="0.0 0.0 0.0" rpy="3.1416 0 0"/>
     <parent link="origin"/>
-    <child link="Index_Base_1"/>
+    <child link="arm_base"/>
   </joint>
 </robot>

File: helix_description/urdf/helix_arm.materials.xacro (robot description, xacro)
@@ -1,3 +1,6 @@
 <?xml version="1.0" ?>
 <robot xmlns:xacro="http://www.ros.org/wiki/xacro" >
+  <material name="white">
+    <color rgba="1 1 1 1"/>
+  </material>
 </robot>

File: helix_description/urdf/helix_arm.xacro (robot description, xacro)
@@ -4,6 +4,54 @@
 <xacro:arg name="mesh_url" default="package://helix_description" />
 <xacro:include filename="$(find helix_description)/urdf/helix_arm.materials.xacro" />
+<link name="arm_base">
+  <visual>
+    <origin xyz="0 0 0" rpy="0 0 0"/>
+      <geometry>
+        <cylinder length="0.005" radius="0.03"/>
+      </geometry>
+    <material name="white"/>
+  </visual>
+</link>
+<link name="seg1_end_link">
+  <visual>
+    <origin xyz="0 0 0" rpy="0 0 0"/>
+      <geometry>
+        <cylinder length="0.005" radius="0.03"/>
+      </geometry>
+    <material name="white"/>
+  </visual>
+</link>
+<joint name="seg1_end_joint" type="floating">
+  <parent link="arm_base"/>
+  <child link="seg1_end_link"/>
+</joint>
+<link name="seg2_end_link">
+  <visual>
+    <origin xyz="0 0 0" rpy="0 0 0"/>
+      <geometry>
+        <cylinder length="0.005" radius="0.03"/>
+      </geometry>
+    <material name="white"/>
+  </visual>
+</link>
+<joint name="seg2_end_joint" type="floating">
+  <parent link="arm_base"/>
+  <child link="seg2_end_link"/>
+</joint>
+<link name="seg3_end_link">
+  <visual>
+    <origin xyz="0 0 0" rpy="0 0 0"/>
+      <geometry>
+        <cylinder length="0.005" radius="0.03"/>
+      </geometry>
+    <material name="white"/>
+  </visual>
+</link>
+<joint name="seg3_end_joint" type="floating">
+  <parent link="arm_base"/>
+  <child link="seg3_end_link"/>
+</joint>
 <!-- Example below for a rigid serial chain. Maybe not relevant at all for flexible Helix arm representation. -->
-<link name="Index_Base_1">
+<!-- <link name="Index_Base_1">
   <inertial>
     <origin xyz="-0.007201714291713072 0.005885230272430774 0.0016787722912366132" rpy="0 0 0"/>
@@ -128,4 +176,4 @@
   <child link="Index_Distal_1"/>
   <axis xyz="-0.99863 0.052336 0.0"/>
-</joint>
+</joint> -->
 </robot>

Commit message: Comment out arm placeholder from URDF

File: helix_description/urdf/helix.urdf.xacro (robot description, xacro)
@@ -3,5 +3,5 @@
   <xacro:include filename="$(find helix_description)/urdf/motor_head.xacro" />
   <xacro:include filename="$(find helix_description)/urdf/helix.ros2_control.xacro" />
-  <xacro:include filename="$(find helix_description)/urdf/helix_arm.xacro"  />
+  <!-- <xacro:include filename="$(find helix_description)/urdf/helix_arm.xacro"  /> -->
   <link name="origin"/>
   <xacro:helix_ros2_control name="helix_ros2_control" />
@@ -9,8 +9,8 @@
     <origin xyz="0 0 0" rpy="0 0 0" />
   </xacro:motor_head>
-  <joint name="arm_to_origin" type="fixed">
+  <!-- <joint name="arm_to_origin" type="fixed">
     <origin xyz="0.0 0.0 0.0" rpy="3.14 0 0"/>
     <parent link="origin"/>
     <child link="Index_Base_1"/>
-  </joint>
+  </joint> -->
 </robot>
