Commit message: Make disc link names numbered instead of lettered

File: helix_description/urdf/helix_arm.xacro (robot description, xacro)
@@ -14,35 +14,35 @@
 <!-- Links for visualisation using floating discs, their transforms can be set manually -->
 <!-- First segment -->
-<joint name="seg1_mid_joint_a" type="floating">
-  <parent link="arm_base"/>
-  <child link="seg1_mid_link_a"/>
-</joint>
-<link name="seg1_mid_link_a">
-  <visual>
-    <origin xyz="0 0 0" rpy="0 0 0"/>
-      <geometry>
-        <cylinder length="0.005" radius="0.03"/>
-      </geometry>
-    <material name="clear"/>
-  </visual>
-</link>
-<joint name="seg1_mid_joint_b" type="floating">
-  <parent link="arm_base"/>
-  <child link="seg1_mid_link_b"/>
-</joint>
-<link name="seg1_mid_link_b">
-  <visual>
-    <origin xyz="0 0 0" rpy="0 0 0"/>
-      <geometry>
-        <cylinder length="0.005" radius="0.03"/>
-      </geometry>
-    <material name="clear"/>
-  </visual>
-</link>
-<joint name="seg1_mid_joint_c" type="floating">
-  <parent link="arm_base"/>
-  <child link="seg1_mid_link_c"/>
-</joint>
-<link name="seg1_mid_link_c">
+<joint name="seg1_mid_joint_1" type="floating">
+  <parent link="arm_base"/>
+  <child link="seg1_mid_link_1"/>
+</joint>
+<link name="seg1_mid_link_1">
+  <visual>
+    <origin xyz="0 0 0" rpy="0 0 0"/>
+      <geometry>
+        <cylinder length="0.005" radius="0.03"/>
+      </geometry>
+    <material name="clear"/>
+  </visual>
+</link>
+<joint name="seg1_mid_joint_2" type="floating">
+  <parent link="arm_base"/>
+  <child link="seg1_mid_link_2"/>
+</joint>
+<link name="seg1_mid_link_2">
+  <visual>
+    <origin xyz="0 0 0" rpy="0 0 0"/>
+      <geometry>
+        <cylinder length="0.005" radius="0.03"/>
+      </geometry>
+    <material name="clear"/>
+  </visual>
+</link>
+<joint name="seg1_mid_joint_3" type="floating">
+  <parent link="arm_base"/>
+  <child link="seg1_mid_link_3"/>
+</joint>
+<link name="seg1_mid_link_3">
   <visual>
     <origin xyz="0 0 0" rpy="0 0 0"/>
@@ -67,87 +67,87 @@
 </link>
 <!-- Second segment -->
-<joint name="seg2_mid_joint_a" type="floating">
-  <parent link="arm_base"/>
-  <child link="seg2_mid_link_a"/>
-</joint>
-<link name="seg2_mid_link_a">
-  <visual>
-    <origin xyz="0 0 0" rpy="0 0 0"/>
-      <geometry>
-        <cylinder length="0.005" radius="0.03"/>
-      </geometry>
-    <material name="clear"/>
-  </visual>
-</link>
-<joint name="seg2_mid_joint_b" type="floating">
-  <parent link="arm_base"/>
-  <child link="seg2_mid_link_b"/>
-</joint>
-<link name="seg2_mid_link_b">
-  <visual>
-    <origin xyz="0 0 0" rpy="0 0 0"/>
-      <geometry>
-        <cylinder length="0.005" radius="0.03"/>
-      </geometry>
-    <material name="clear"/>
-  </visual>
-</link>
-<joint name="seg2_mid_joint_c" type="floating">
-  <parent link="arm_base"/>
-  <child link="seg2_mid_link_c"/>
-</joint>
-<link name="seg2_mid_link_c">
-  <visual>
-    <origin xyz="0 0 0" rpy="0 0 0"/>
-      <geometry>
-        <cylinder length="0.005" radius="0.03"/>
-      </geometry>
-    <material name="clear"/>
-  </visual>
-</link>
-<joint name="seg2_mid_joint_d" type="floating">
-  <parent link="arm_base"/>
-  <child link="seg2_mid_link_d"/>
-</joint>
-<link name="seg2_mid_link_d">
-  <visual>
-    <origin xyz="0 0 0" rpy="0 0 0"/>
-      <geometry>
-        <cylinder length="0.005" radius="0.03"/>
-      </geometry>
-    <material name="clear"/>
-  </visual>
-</link>
-<joint name="seg2_mid_joint_e" type="floating">
-  <parent link="arm_base"/>
-  <child link="seg2_mid_link_e"/>
-</joint>
-<link name="seg2_mid_link_e">
-  <visual>
-    <origin xyz="0 0 0" rpy="0 0 0"/>
-      <geometry>
-        <cylinder length="0.005" radius="0.03"/>
-      </geometry>
-    <material name="clear"/>
-  </visual>
-</link>
-<joint name="seg2_mid_joint_f" type="floating">
-  <parent link="arm_base"/>
-  <child link="seg2_mid_link_f"/>
-</joint>
-<link name="seg2_mid_link_f">
-  <visual>
-    <origin xyz="0 0 0" rpy="0 0 0"/>
-      <geometry>
-        <cylinder length="0.005" radius="0.03"/>
-      </geometry>
-    <material name="clear"/>
-  </visual>
-</link>
-<joint name="seg2_mid_joint_g" type="floating">
-  <parent link="arm_base"/>
-  <child link="seg2_mid_link_g"/>
-</joint>
-<link name="seg2_mid_link_g">
+<joint name="seg2_mid_joint_1" type="floating">
+  <parent link="arm_base"/>
+  <child link="seg2_mid_link_1"/>
+</joint>
+<link name="seg2_mid_link_1">
+  <visual>
+    <origin xyz="0 0 0" rpy="0 0 0"/>
+      <geometry>
+        <cylinder length="0.005" radius="0.03"/>
+      </geometry>
+    <material name="clear"/>
+  </visual>
+</link>
+<joint name="seg2_mid_joint_2" type="floating">
+  <parent link="arm_base"/>
+  <child link="seg2_mid_link_2"/>
+</joint>
+<link name="seg2_mid_link_2">
+  <visual>
+    <origin xyz="0 0 0" rpy="0 0 0"/>
+      <geometry>
+        <cylinder length="0.005" radius="0.03"/>
+      </geometry>
+    <material name="clear"/>
+  </visual>
+</link>
+<joint name="seg2_mid_joint_3" type="floating">
+  <parent link="arm_base"/>
+  <child link="seg2_mid_link_3"/>
+</joint>
+<link name="seg2_mid_link_3">
+  <visual>
+    <origin xyz="0 0 0" rpy="0 0 0"/>
+      <geometry>
+        <cylinder length="0.005" radius="0.03"/>
+      </geometry>
+    <material name="clear"/>
+  </visual>
+</link>
+<joint name="seg2_mid_joint_4" type="floating">
+  <parent link="arm_base"/>
+  <child link="seg2_mid_link_4"/>
+</joint>
+<link name="seg2_mid_link_4">
+  <visual>
+    <origin xyz="0 0 0" rpy="0 0 0"/>
+      <geometry>
+        <cylinder length="0.005" radius="0.03"/>
+      </geometry>
+    <material name="clear"/>
+  </visual>
+</link>
+<joint name="seg2_mid_joint_5" type="floating">
+  <parent link="arm_base"/>
+  <child link="seg2_mid_link_5"/>
+</joint>
+<link name="seg2_mid_link_5">
+  <visual>
+    <origin xyz="0 0 0" rpy="0 0 0"/>
+      <geometry>
+        <cylinder length="0.005" radius="0.03"/>
+      </geometry>
+    <material name="clear"/>
+  </visual>
+</link>
+<joint name="seg2_mid_joint_6" type="floating">
+  <parent link="arm_base"/>
+  <child link="seg2_mid_link_6"/>
+</joint>
+<link name="seg2_mid_link_6">
+  <visual>
+    <origin xyz="0 0 0" rpy="0 0 0"/>
+      <geometry>
+        <cylinder length="0.005" radius="0.03"/>
+      </geometry>
+    <material name="clear"/>
+  </visual>
+</link>
+<joint name="seg2_mid_joint_7" type="floating">
+  <parent link="arm_base"/>
+  <child link="seg2_mid_link_7"/>
+</joint>
+<link name="seg2_mid_link_7">
   <visual>
     <origin xyz="0 0 0" rpy="0 0 0"/>
@@ -172,87 +172,87 @@
 </link>
 <!-- Third segment -->
-<joint name="seg3_mid_joint_a" type="floating">
-  <parent link="arm_base"/>
-  <child link="seg3_mid_link_a"/>
-</joint>
-<link name="seg3_mid_link_a">
-  <visual>
-    <origin xyz="0 0 0" rpy="0 0 0"/>
-      <geometry>
-        <cylinder length="0.005" radius="0.03"/>
-      </geometry>
-    <material name="clear"/>
-  </visual>
-</link>
-<joint name="seg3_mid_joint_b" type="floating">
-  <parent link="arm_base"/>
-  <child link="seg3_mid_link_b"/>
-</joint>
-<link name="seg3_mid_link_b">
-  <visual>
-    <origin xyz="0 0 0" rpy="0 0 0"/>
-      <geometry>
-        <cylinder length="0.005" radius="0.03"/>
-      </geometry>
-    <material name="clear"/>
-  </visual>
-</link>
-<joint name="seg3_mid_joint_c" type="floating">
-  <parent link="arm_base"/>
-  <child link="seg3_mid_link_c"/>
-</joint>
-<link name="seg3_mid_link_c">
-  <visual>
-    <origin xyz="0 0 0" rpy="0 0 0"/>
-      <geometry>
-        <cylinder length="0.005" radius="0.03"/>
-      </geometry>
-    <material name="clear"/>
-  </visual>
-</link>
-<joint name="seg3_mid_joint_d" type="floating">
-  <parent link="arm_base"/>
-  <child link="seg3_mid_link_d"/>
-</joint>
-<link name="seg3_mid_link_d">
-  <visual>
-    <origin xyz="0 0 0" rpy="0 0 0"/>
-      <geometry>
-        <cylinder length="0.005" radius="0.03"/>
-      </geometry>
-    <material name="clear"/>
-  </visual>
-</link>
-<joint name="seg3_mid_joint_e" type="floating">
-  <parent link="arm_base"/>
-  <child link="seg3_mid_link_e"/>
-</joint>
-<link name="seg3_mid_link_e">
-  <visual>
-    <origin xyz="0 0 0" rpy="0 0 0"/>
-      <geometry>
-        <cylinder length="0.005" radius="0.03"/>
-      </geometry>
-    <material name="clear"/>
-  </visual>
-</link>
-<joint name="seg3_mid_joint_f" type="floating">
-  <parent link="arm_base"/>
-  <child link="seg3_mid_link_f"/>
-</joint>
-<link name="seg3_mid_link_f">
-  <visual>
-    <origin xyz="0 0 0" rpy="0 0 0"/>
-      <geometry>
-        <cylinder length="0.005" radius="0.03"/>
-      </geometry>
-    <material name="clear"/>
-  </visual>
-</link>
-<joint name="seg3_mid_joint_g" type="floating">
-  <parent link="arm_base"/>
-  <child link="seg3_mid_link_g"/>
-</joint>
-<link name="seg3_mid_link_g">
+<joint name="seg3_mid_joint_1" type="floating">
+  <parent link="arm_base"/>
+  <child link="seg3_mid_link_1"/>
+</joint>
+<link name="seg3_mid_link_1">
+  <visual>
+    <origin xyz="0 0 0" rpy="0 0 0"/>
+      <geometry>
+        <cylinder length="0.005" radius="0.03"/>
+      </geometry>
+    <material name="clear"/>
+  </visual>
+</link>
+<joint name="seg3_mid_joint_2" type="floating">
+  <parent link="arm_base"/>
+  <child link="seg3_mid_link_2"/>
+</joint>
+<link name="seg3_mid_link_2">
+  <visual>
+    <origin xyz="0 0 0" rpy="0 0 0"/>
+      <geometry>
+        <cylinder length="0.005" radius="0.03"/>
+      </geometry>
+    <material name="clear"/>
+  </visual>
+</link>
+<joint name="seg3_mid_joint_3" type="floating">
+  <parent link="arm_base"/>
+  <child link="seg3_mid_link_3"/>
+</joint>
+<link name="seg3_mid_link_3">
+  <visual>
+    <origin xyz="0 0 0" rpy="0 0 0"/>
+      <geometry>
+        <cylinder length="0.005" radius="0.03"/>
+      </geometry>
+    <material name="clear"/>
+  </visual>
+</link>
+<joint name="seg3_mid_joint_4" type="floating">
+  <parent link="arm_base"/>
+  <child link="seg3_mid_link_4"/>
+</joint>
+<link name="seg3_mid_link_4">
+  <visual>
+    <origin xyz="0 0 0" rpy="0 0 0"/>
+      <geometry>
+        <cylinder length="0.005" radius="0.03"/>
+      </geometry>
+    <material name="clear"/>
+  </visual>
+</link>
+<joint name="seg3_mid_joint_5" type="floating">
+  <parent link="arm_base"/>
+  <child link="seg3_mid_link_5"/>
+</joint>
+<link name="seg3_mid_link_5">
+  <visual>
+    <origin xyz="0 0 0" rpy="0 0 0"/>
+      <geometry>
+        <cylinder length="0.005" radius="0.03"/>
+      </geometry>
+    <material name="clear"/>
+  </visual>
+</link>
+<joint name="seg3_mid_joint_6" type="floating">
+  <parent link="arm_base"/>
+  <child link="seg3_mid_link_6"/>
+</joint>
+<link name="seg3_mid_link_6">
+  <visual>
+    <origin xyz="0 0 0" rpy="0 0 0"/>
+      <geometry>
+        <cylinder length="0.005" radius="0.03"/>
+      </geometry>
+    <material name="clear"/>
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