Commit message: Add a controller for gripper motor

File: helix_description/urdf/motor_head.xacro (robot description, xacro)
@@ -188,4 +188,21 @@
     </visual>
   </link>
+  <!-- Gripper Joint -->
+  <joint name="joint_gripper" type="continuous">
+    <parent link="base"/>
+    <child link="link_gripper"/>
+    <origin xyz="0 0 0.2" rpy="0 0 0"/>
+    <axis xyz="1 0 0"/>
+  </joint>
+   <!-- Gripper Link -->
+  <link name="link_gripper">
+    <visual>
+      <origin xyz="0 0 0" rpy="0 1.57 0"/>
+      <geometry>
+        <cylinder length="0.015" radius="0.02"/>
+      </geometry>
+      <material name="black"/>
+    </visual>
+  </link>
 </xacro:macro>
 </robot>
