Commit message: Merge helix_description seb to max

File: helix_description/urdf/helix.ros2_control.xacro (robot description, xacro)
@@ -1,104 +1,82 @@
 <?xml version="1.0"?>
 <robot xmlns:xacro="http://www.ros.org/wiki/xacro">
-  <xacro:macro name="dynamixel_block_ros2_control" params="name">
+  <xacro:macro name="helix_ros2_control" params="name">
     <ros2_control name="${name}" type="system">
       <hardware>
         <plugin>dynamixel_hardware/DynamixelHardware</plugin>
         <param name="usb_port">/dev/ttyUSB0</param>
-        <param name="baud_rate">3000000</param>
+        <param name="baud_rate">1000000</param>
         <param name="use_dummy">true</param>
       </hardware>
-      <joint name="dynamixel0">
+      <joint name="joint0">
+        <!-- id is Dynamixel Motor ID -->
         <param name="id">0</param>
         <command_interface name="position"/>
-        <command_interface name="velocity"/>
+        <!-- effort interface for current control -->
+        <command_interface name="effort"/>
         <state_interface name="position"/>
         <state_interface name="velocity"/>
         <state_interface name="effort"/>
       </joint>
-      <joint name="dynamixel1">
+      <joint name="joint1">
         <param name="id">1</param>
         <command_interface name="position"/>
-        <command_interface name="velocity"/>
+        <command_interface name="effort"/>
         <state_interface name="position"/>
         <state_interface name="velocity"/>
         <state_interface name="effort"/>
       </joint>
-      <joint name="dynamixel2">
+      <joint name="joint2">
         <param name="id">2</param>
         <command_interface name="position"/>
-        <command_interface name="velocity"/>
+        <command_interface name="effort"/>
         <state_interface name="position"/>
         <state_interface name="velocity"/>
         <state_interface name="effort"/>
       </joint>
-      <joint name="dynamixel3">
+      <joint name="joint3">
         <param name="id">3</param>
         <command_interface name="position"/>
-        <command_interface name="velocity"/>
+        <command_interface name="effort"/>
         <state_interface name="position"/>
         <state_interface name="velocity"/>
         <state_interface name="effort"/>
       </joint>
-      <joint name="dynamixel4">
+      <joint name="joint4">
         <param name="id">4</param>
         <command_interface name="position"/>
-        <command_interface name="velocity"/>
+        <command_interface name="effort"/>
         <state_interface name="position"/>
         <state_interface name="velocity"/>
         <state_interface name="effort"/>
       </joint>
-      <joint name="dynamixel5">
+      <joint name="joint5">
         <param name="id">5</param>
         <command_interface name="position"/>
-        <command_interface name="velocity"/>
+        <command_interface name="effort"/>
         <state_interface name="position"/>
         <state_interface name="velocity"/>
         <state_interface name="effort"/>
       </joint>
-      <joint name="dynamixel6">
+      <joint name="joint6">
         <param name="id">6</param>
         <command_interface name="position"/>
-        <command_interface name="velocity"/>
+        <command_interface name="effort"/>
         <state_interface name="position"/>
         <state_interface name="velocity"/>
         <state_interface name="effort"/>
       </joint>
-      <joint name="dynamixel7">
+      <joint name="joint7">
         <param name="id">7</param>
         <command_interface name="position"/>
-        <command_interface name="velocity"/>
+        <command_interface name="effort"/>
         <state_interface name="position"/>
         <state_interface name="velocity"/>
         <state_interface name="effort"/>
       </joint>
-      <joint name="dynamixel8">
+      <joint name="joint8">
         <param name="id">8</param>
         <command_interface name="position"/>
-        <command_interface name="velocity"/>
-        <state_interface name="position"/>
-        <state_interface name="velocity"/>
-        <state_interface name="effort"/>
-      </joint>
-      <joint name="dynamixel9">
-        <param name="id">9</param>
-        <command_interface name="position"/>
-        <command_interface name="velocity"/>
-        <state_interface name="position"/>
-        <state_interface name="velocity"/>
-        <state_interface name="effort"/>
-      </joint>
-      <joint name="dynamixel10">
-        <param name="id">10</param>
-        <command_interface name="position"/>
-        <command_interface name="velocity"/>
-        <state_interface name="position"/>
-        <state_interface name="velocity"/>
-        <state_interface name="effort"/>
-      </joint>
-      <joint name="dynamixel11">
-        <param name="id">11</param>
-        <command_interface name="position"/>
-        <command_interface name="velocity"/>
+        <command_interface name="effort"/>
         <state_interface name="position"/>
         <state_interface name="velocity"/>

File: helix_description/urdf/helix.urdf.xacro (robot description, xacro)
@@ -1,16 +1,17 @@
 <?xml version="1.0"?>
 <robot name="helix_description" xmlns:xacro="http://ros.org/wiki/xacro">
-  <xacro:include filename="$(find helix_description)/urdf/dynamixel_block.xacro" />
-  <xacro:include filename="$(find helix_description)/urdf/dynamixel_block.ros2_control.xacro" />
-  <xacro:include filename="$(find helix_description)/urdf/helix.xacro"  />
+  <xacro:include filename="$(find helix_description)/urdf/motor_head.xacro" />
+  <xacro:include filename="$(find helix_description)/urdf/helix.ros2_control.xacro" />
+  <!-- <xacro:include filename="$(find helix_description)/urdf/helix.xacro"  /> -->
   <link name="world"/>
-  <xacro:dynamixel_block_ros2_control name="dynamixel_block_ros2_control" />
-  <xacro:dynamixel_block parent="world">
+  <xacro:helix_ros2_control name="helix_ros2_control" />
+  <xacro:motor_head parent="world">
     <origin xyz="0 0 0" rpy="0 0 0" />
-  </xacro:dynamixel_block>
-  <joint name="hand_to_world" type="fixed">
+  </xacro:motor_head>
+<!--
+  <joint name="motor_head_to_world" type="fixed">
     <origin xyz="0.0 0.0 0.1" rpy="0 0 0"/>
     <parent link="world"/>
-    <child link="base_link"/>
-  </joint>
+    <child link="base"/>
+  </joint> -->
 </robot>

File: helix_description/urdf/motor_head.materials.xacro (robot description, xacro)
@@ -1,9 +1,9 @@
 <?xml version="1.0"?>
 <robot>
-  <material name="dynamixel_body">
-    <color rgba="0.500 0.500 0.500 1.000"/>
-  </material>
   <material name="dynamixel_horn">
     <color rgba="0.7 0.6 0.0 1.000"/>
   </material>
+  <material name='clear'>
+    <color rgba="0.2 0.2 0.2 0.2"/>
+  </material>
 </robot>

Commit message: Tested Extended Position mode with hardware

File: helix_description/urdf/helix.ros2_control.xacro (robot description, xacro)
@@ -7,5 +7,5 @@
         <param name="usb_port">/dev/ttyUSB0</param>
         <param name="baud_rate">1000000</param>
-        <param name="use_dummy">true</param>
+        <!-- <param name="use_dummy">true</param> -->
       </hardware>
       <joint name="joint0">

File: helix_description/urdf/motor_head.xacro (robot description, xacro)
@@ -36,11 +36,9 @@
   </link>
   <!-- Joint 0 -->
-  <!-- TODO check changing to continuous, removing limits -->
-  <joint name="joint0" type="revolute">
+  <joint name="joint0" type="continuous">
     <parent link="base"/>
     <child link="link0"/>
     <origin xyz="-0.043 0.025 0.12" rpy="0 0 4.2"/>
     <axis xyz="1 0 0"/>
-    <limit velocity="4.8" effort="1" lower="-3.0" upper="3.0" />
   </joint>
    <!-- Link 0 -->
@@ -55,10 +53,9 @@
   </link>
   <!-- Joint 1 -->
-  <joint name="joint1" type="revolute">
+  <joint name="joint1" type="continuous">
     <parent link="base"/>
     <child link="link1"/>
     <origin xyz="0 -0.05 0.12" rpy="0 0 0"/>
     <axis xyz="1 0 0"/>
-    <limit velocity="4.8" effort="1" lower="-3.0" upper="3.0" />
   </joint>
    <!-- Link 1 -->
@@ -73,10 +70,10 @@
   </link>
   <!-- Joint 2 -->
-  <joint name="joint2" type="revolute">
+  <joint name="joint2" type="continuous">
     <parent link="base"/>
     <child link="link2"/>
     <origin xyz="0.043 0.025 0.12" rpy="0 0 2.1"/>
     <axis xyz="1 0 0"/>
-    <limit velocity="4.8" effort="1" lower="-3.0" upper="3.0" />
+    continuous
   </joint>
    <!-- Link 2 -->
@@ -91,10 +88,9 @@
   </link>
   <!-- Joint 3 -->
-  <joint name="joint3" type="revolute">
+  <joint name="joint3" type="continuous">
     <parent link="base"/>
     <child link="link3"/>
     <origin xyz="0.16 0 0.025" rpy="0 0 0"/>
     <axis xyz="1 0 0"/>
-    <limit velocity="4.8" effort="1" lower="-3.0" upper="3.0" />
   </joint>
    <!-- Link 3 -->
@@ -109,10 +105,9 @@
   </link>
   <!-- Joint 4 -->
-  <joint name="joint4" type="revolute">
+  <joint name="joint4" type="continuous">
     <parent link="base"/>
     <child link="link4"/>
     <origin xyz="-0.08 0.138 0.025" rpy="0 0 2.1"/>
     <axis xyz="1 0 0"/>
-    <limit velocity="4.8" effort="1" lower="-3.0" upper="3.0" />
   </joint>
    <!-- Link 4 -->
@@ -127,10 +122,9 @@
   </link>
   <!-- Joint 5 -->
-  <joint name="joint5" type="revolute">
+  <joint name="joint5" type="continuous">
     <parent link="base"/>
     <child link="link5"/>
     <origin xyz="-0.08 -0.138 0.025" rpy="0 0 4.2"/>
     <axis xyz="1 0 0"/>
-    <limit velocity="4.8" effort="1" lower="-3.0" upper="3.0" />
   </joint>
    <!-- Link 5 -->
@@ -145,10 +139,9 @@
   </link>
   <!-- Joint 6 -->
-  <joint name="joint6" type="revolute">
+  <joint name="joint6" type="continuous">
     <parent link="base"/>
     <child link="link6"/>
     <origin xyz="0.08 -0.138 0.025" rpy="0 0 5.2"/>
     <axis xyz="1 0 0"/>
-    <limit velocity="4.8" effort="1" lower="-3.0" upper="3.0" />
   </joint>
    <!-- Link 6 -->
@@ -163,10 +156,9 @@
   </link>
   <!-- Joint 7 -->
-  <joint name="joint7" type="revolute">
+  <joint name="joint7" type="continuous">
     <parent link="base"/>
     <child link="link7"/>
     <origin xyz="0.08 0.138 0.025" rpy="0 0 1.0"/>
     <axis xyz="1 0 0"/>
-    <limit velocity="4.8" effort="1" lower="-3.0" upper="3.0" />
   </joint>
    <!-- Link 7 -->
@@ -181,10 +173,9 @@
   </link>
   <!-- Joint 8 -->
-  <joint name="joint8" type="revolute">
+  <joint name="joint8" type="continuous">
     <parent link="base"/>
     <child link="link8"/>
     <origin xyz="-0.16 0 0.025" rpy="0 0 3.1"/>
     <axis xyz="1 0 0"/>
-    <limit velocity="4.8" effort="1" lower="-3.0" upper="3.0" />
   </joint>
    <!-- Link 8 -->

Commit message: Add in gripper joint ros_control definition that got deleted

File: helix_description/urdf/helix.ros2_control.xacro (robot description, xacro)
@@ -83,4 +83,12 @@
         <state_interface name="effort"/>
       </joint>
+      <joint name="joint_gripper">
+        <param name="id">9</param>
+        <command_interface name="position"/>
+        <command_interface name="effort"/>
+        <state_interface name="position"/>
+        <state_interface name="velocity"/>
+        <state_interface name="effort"/>
+      </joint>
     </ros2_control>
   </xacro:macro>

Commit message: Remove gripper controller

File: helix_description/urdf/helix.ros2_control.xacro (robot description, xacro)
@@ -83,12 +83,4 @@
         <state_interface name="effort"/>
       </joint>
-      <joint name="joint_gripper">
-        <param name="id">9</param>
-        <command_interface name="position"/>
-        <command_interface name="effort"/>
-        <state_interface name="position"/>
-        <state_interface name="velocity"/>
-        <state_interface name="effort"/>
-      </joint>
     </ros2_control>
   </xacro:macro>

File: helix_description/urdf/motor_head.xacro (robot description, xacro)
@@ -188,21 +188,4 @@
     </visual>
   </link>
-  <!-- Gripper Joint -->
-  <joint name="joint_gripper" type="continuous">
-    <parent link="base"/>
-    <child link="link_gripper"/>
-    <origin xyz="0 0 0.2" rpy="0 0 0"/>
-    <axis xyz="1 0 0"/>
-  </joint>
-   <!-- Gripper Link -->
-  <link name="link_gripper">
-    <visual>
-      <origin xyz="0 0 0" rpy="0 1.57 0"/>
-      <geometry>
-        <cylinder length="0.015" radius="0.02"/>
-      </geometry>
-      <material name="black"/>
-    </visual>
-  </link>
 </xacro:macro>
 </robot>

Commit message: Add gripper motor controller with position mode only

File: helix_description/urdf/helix.ros2_control.xacro (robot description, xacro)
@@ -83,4 +83,11 @@
         <state_interface name="effort"/>
       </joint>
+      <joint name="joint_gripper">
+        <param name="id">9</param>
+        <command_interface name="position"/>
+        <state_interface name="position"/>
+        <state_interface name="velocity"/>
+        <state_interface name="effort"/>
+      </joint>
     </ros2_control>
   </xacro:macro>

Commit message: This is what should be removed to allow the system to run without the gripper motor connected

File: helix_description/urdf/helix.ros2_control.xacro (robot description, xacro)
@@ -83,5 +83,5 @@
         <state_interface name="effort"/>
       </joint>
-      <joint name="joint_gripper">
+      <!-- <joint name="joint_gripper">
         <param name="id">9</param>
         <command_interface name="position"/>
@@ -89,5 +89,5 @@
         <state_interface name="velocity"/>
         <state_interface name="effort"/>
-      </joint>
+      </joint> -->
     </ros2_control>
   </xacro:macro>
